File: power.sch (KiCad schematic (older format))
At the start: 30 parts

Commit message: Use LT8609 for power supply.
Parts:
- removed C?: CP, symbol CP
- removed C? (x3): 100n, symbol C
- removed C? (x2): C, symbol C
- removed C?: 10u, symbol C
- removed C?: 22u, symbol C
- removed D?: B130LAW-7-F, SOD-123, symbol D_Schottky
- removed L?: L, symbol INDUCTOR
- removed L?: 10uH 0.045Ohm, symbol INDUCTOR
- removed R? (x5): R, symbol R
- removed R?: 10k2, symbol R
- removed R?: 1k96, symbol R
- removed U?: TPS54233, SOIC8, symbol TPS54233
- removed U?: TPS560200, SOT23, symbol TPS560200
- added C? (x2): 100n X7R, symbol C
- added C? (x2): 10p, symbol C
- added C? (x3): 22µ, symbol C
- added C? (x2): 1µ, symbol C
- added C?: 100n, symbol C
- added C? (x2): 10n, symbol C
- added L? (x2): 3µ3, symbol INDUCTOR
- added R? (x2): 1M, symbol R
- added R?: 309k, symbol R
- added R? (x2): 60k4, symbol R
- added R? (x2): 330k, symbol R
- added R? (x2): 47k, symbol R
- added R?: 178k, symbol R
- added R? (x2): 100k, symbol R
- added U? (x2): LT8609, symbol LT8609
Connections:
- wire segments 82 -> 139
Other:
- moved on the sheet: C?, D?, R?

Commit message: Reverse voltage protection.
Parts:
- added C?: 100n, symbol C
- added D?: 10V, SOD-323, symbol ZENER
- added Q?: DMP6050SFG, POWERDI3333-8, symbol DMP6050SFG
- added R?: 100k, symbol R
Connections:
- wire segments 139 -> 115
Other:
- note added: "12..24 V"
- moved on the sheet: C?, D?, R?

Commit message: changes on power supply; start redesign 3.3V rail
Parts:
- added L?: 1µH, symbol INDUCTOR
- added U?: LTC3564, symbol LTC3564
Connections:
- wire segments 115 -> 119
Other:
- note added: "5V 2A"
Changed lines of the file:
@@
 $EndComp
 $Comp
-L VBAT #PWR?
+L VBAT #PWR01
 U 1 1 562B8E65
 P 2050 5450
-F 0 "#PWR?" H 2050 5300 50  0001 C CNN
+F 0 "#PWR01" H 2050 5300 50  0001 C CNN
 F 1 "VBAT" H 2050 5590 50  0000 C CNN
 F 2 "" H 2050 5450 60  0000 C CNN
@@
 $EndComp
 $Comp
-L GND #PWR?
+L GND #PWR02
 U 1 1 562B8F95
 P 1200 7000
-F 0 "#PWR?" H 1200 6750 50  0001 C CNN
+F 0 "#PWR02" H 1200 6750 50  0001 C CNN
 F 1 "GND" H 1200 6850 50  0000 C CNN
 F 2 "" H 1200 7000 60  0000 C CNN
@@
 $EndComp
 $Comp
-L GND #PWR?
+L GND #PWR03
 U 1 1 562B96C2
 P 2050 7000
-F 0 "#PWR?" H 2050 6750 50  0001 C CNN
+F 0 "#PWR03" H 2050 6750 50  0001 C CNN
 F 1 "GND" H 2050 6850 50  0000 C CNN
 F 2 "" H 2050 7000 60  0000 C CNN
@@
 $EndComp
 $Comp
-L +5V #PWR?
+L +5V #PWR04
 U 1 1 562BA71E
 P 10250 1400
-F 0 "#PWR?" H 10250 1250 50  0001 C CNN
+F 0 "#PWR04" H 10250 1250 50  0001 C CNN
 F 1 "+5V" H 10250 1540 50  0000 C CNN
 F 2 "" H 10250 1400 60  0000 C CNN
@@
 $EndComp
 $Comp
-L VIN #PWR?
+L VIN #PWR05
 U 1 1 562BB258
 P 750 1250
-F 0 "#PWR?" H 750 1100 50  0001 C CNN
+F 0 "#PWR05" H 750 1100 50  0001 C CNN
 F 1 "VIN" H 750 1390 50  0000 C CNN
 F 2 "" H 750 1250 60  0000 C CNN
@@
 $EndComp
 $Comp
-L GND #PWR?
+L GND #PWR06
 U 1 1 562BC4C3
 P -1050 -1350
-F 0 "#PWR?" H -1050 -1600 50  0001 C CNN
+F 0 "#PWR06" H -1050 -1600 50  0001 C CNN
 F 1 "GND" H -1050 -1500 50  0000 C CNN
 F 2 "" H -1050 -1350 60  0000 C CNN
@@
 $EndComp
 $Comp
-L GND #PWR?
+L GND #PWR07
 U 1 1 562BD4E1
 P -200 -1350
-F 0 "#PWR?" H -200 -1600 50  0001 C CNN
+F 0 "#PWR07" H -200 -1600 50  0001 C CNN
 F 1 "GND" H -200 -1500 50  0000 C CNN
 F 2 "" H -200 -1350 60  0000 C CNN
@@
 $EndComp
 $Comp
-L GND #PWR?
+L GND #PWR08
 U 1 1 562BEC1D
 P -1400 -1350
-F 0 "#PWR?" H -1400 -1600 50  0001 C CNN
+F 0 "#PWR08" H -1400 -1600 50  0001 C CNN
 F 1 "GND" H -1400 -1500 50  0000 C CNN
 F 2 "" H -1400 -1350 60  0000 C CNN
@@
 $EndComp
 $Comp
-L +3.3V #PWR?
+L +3.3V #PWR09
 U 1 1 562C0A20
 P 1200 5450
-F 0 "#PWR?" H 1200 5300 50  0001 C CNN
+F 0 "#PWR09" H 1200 5300 50  0001 C CNN
 F 1 "+3.3V" H 1200 5590 50  0000 C CNN
 F 2 "" H 1200 5450 60  0000 C CNN
@@
 Connection ~ 9200 1600
 $Comp
-L GND #PWR?
+L GND #PWR010
 U 1 1 5634F800
 P 9200 2850
-F 0 "#PWR?" H 9200 2600 50  0001 C CNN
+F 0 "#PWR010" H 9200 2600 50  0001 C CNN
 F 1 "GND" H 9200 2700 50  0000 C CNN
 F 2 "" H 9200 2850 60  0000 C CNN
@@
 Connection ~ 7800 2300
 $Comp
-L GND #PWR?
+L GND #PWR011
 U 1 1 5634FAFB
 P 7800 2850
-F 0 "#PWR?" H 7800 2600 50  0001 C CNN
+F 0 "#PWR011" H 7800 2600 50  0001 C CNN
 F 1 "GND" H 7800 2700 50  0000 C CNN
 F 2 "" H 7800 2850 60  0000 C CNN
@@
 $EndComp
 $Comp
-L GND #PWR?
+L GND #PWR012
 U 1 1 5634FB75
 P 6500 2850
-F 0 "#PWR?" H 6500 2600 50  0001 C CNN
+F 0 "#PWR012" H 6500 2600 50  0001 C CNN
 F 1 "GND" H 6500 2700 50  0000 C CNN
 F 2 "" H 6500 2850 60  0000 C CNN
@@
 	5700 2400 5800 2400
 $Comp
-L GND #PWR?
+L GND #PWR013
 U 1 1 563500D2
 P 5700 2900
-F 0 "#PWR?" H 5700 2650 50  0001 C CNN
+F 0 "#PWR013" H 5700 2650 50  0001 C CNN
 F 1 "GND" H 5700 2750 50  0000 C CNN
 F 2 "" H 5700 2900 60  0000 C CNN
@@
 	5700 2900 5700 2800
 $Comp
-L GND #PWR?
+L GND #PWR014
 U 1 1 5635050E
 P 4950 2900
-F 0 "#PWR?" H 4950 2650 50  0001 C CNN
+F 0 "#PWR014" H 4950 2650 50  0001 C CNN
 F 1 "GND" H 4950 2750 50  0000 C CNN
 F 2 "" H 4950 2900 60  0000 C CNN
@@
 	400  -2350 400  -2750
 $Comp
-L GND #PWR?
+L GND #PWR015
 U 1 1 563511D1
 P 400 -1250
-F 0 "#PWR?" H 400 -1500 50  0001 C CNN
+F 0 "#PWR015" H 400 -1500 50  0001 C CNN
 F 1 "GND" H 400 -1400 50  0000 C CNN
 F 2 "" H 400 -1250 60  0000 C CNN
@@
 $EndComp
 $Comp
-L GND #PWR?
+L GND #PWR016
 U 1 1 56351E27
 P 4200 2900
-F 0 "#PWR?" H 4200 2650 50  0001 C CNN
+F 0 "#PWR016" H 4200 2650 50  0001 C CNN
 F 1 "GND" H 4200 2750 50  0000 C CNN
 F 2 "" H 4200 2900 60  0000 C CNN
@@
 	5300 2200 5300 2500
 $Comp
-L GND #PWR?
+L GND #PWR017
 U 1 1 5635362E
 P 5300 2900
-F 0 "#PWR?" H 5300 2650 50  0001 C CNN
+F 0 "#PWR017" H 5300 2650 50  0001 C CNN
 F 1 "GND" H 5300 2750 50  0000 C CNN
 F 2 "" H 5300 2900 60  0000 C CNN
@@
 $EndComp
 $Comp
-L GND #PWR?
+L GND #PWR018
 U 1 1 56353BBC
 P 4500 2900
-F 0 "#PWR?" H 4500 2650 50  0001 C CNN
+F 0 "#PWR018" H 4500 2650 50  0001 C CNN
 F 1 "GND" H 4500 2750 50  0000 C CNN
 F 2 "" H 4500 2900 60  0000 C CNN
@@
 Connection ~ 9200 4600
 $Comp
-L GND #PWR?
+L GND #PWR019
 U 1 1 56355C5D
 P 9200 5850
-F 0 "#PWR?" H 9200 5600 50  0001 C CNN
+F 0 "#PWR019" H 9200 5600 50  0001 C CNN
 F 1 "GND" H 9200 5700 50  0000 C CNN
 F 2 "" H 9200 5850 60  0000 C CNN
@@
 Connection ~ 7800 5300
 $Comp
-L GND #PWR?
+L GND #PWR020
 U 1 1 56355C6C
 P 7800 5850
-F 0 "#PWR?" H 7800 5600 50  0001 C CNN
+F 0 "#PWR020" H 7800 5600 50  0001 C CNN
 F 1 "GND" H 7800 5700 50  0000 C CNN
 F 2 "" H 7800 5850 60  0000 C CNN
@@
 	5700 5400 5800 5400
 $Comp
-L GND #PWR?
+L GND #PWR021
 U 1 1 56356A63
 P 5700 5900
-F 0 "#PWR?" H 5700 5650 50  0001 C CNN
+F 0 "#PWR021" H 5700 5650 50  0001 C CNN
 F 1 "GND" H 5700 5750 50  0000 C CNN
 F 2 "" H 5700 5900 60  0000 C CNN
@@
 	5700 5900 5700 5800
 $Comp
-L GND #PWR?
+L GND #PWR022
 U 1 1 56356A6C
 P 4950 5900
-F 0 "#PWR?" H 4950 5650 50  0001 C CNN
+F 0 "#PWR022" H 4950 5650 50  0001 C CNN
 F 1 "GND" H 4950 5750 50  0000 C CNN
 F 2 "" H 4950 5900 60  0000 C CNN
@@
 	5300 5200 5300 5500
 $Comp
-L GND #PWR?
+L GND #PWR023
 U 1 1 56356A7D
 P 5300 5900
-F 0 "#PWR?" H 5300 5650 50  0001 C CNN
+F 0 "#PWR023" H 5300 5650 50  0001 C CNN
 F 1 "GND" H 5300 5750 50  0000 C CNN
 F 2 "" H 5300 5900 60  0000 C CNN
@@
 $EndComp
 $Comp
-L GND #PWR?
+L GND #PWR024
 U 1 1 56356A90
 P 4500 5900
-F 0 "#PWR?" H 4500 5650 50  0001 C CNN
+F 0 "#PWR024" H 4500 5650 50  0001 C CNN
 F 1 "GND" H 4500 5750 50  0000 C CNN
 F 2 "" H 4500 5900 60  0000 C CNN
@@
 	4950 5000 5800 5000
 $Comp
-L GND #PWR?
+L GND #PWR025
 U 1 1 563589D3
 P 6500 5900
-F 0 "#PWR?" H 6500 5650 50  0001 C CNN
+F 0 "#PWR025" H 6500 5650 50  0001 C CNN
 F 1 "GND" H 6500 5750 50  0000 C CNN
 F 2 "" H 6500 5900 60  0000 C CNN
@@
 	6500 5900 6500 5700
 $Comp
-L +3.3V #PWR?
+L +3.3V #PWR026
 U 1 1 56358F87
 P 10250 4350
-F 0 "#PWR?" H 10250 4200 50  0001 C CNN
+F 0 "#PWR026" H 10250 4200 50  0001 C CNN
 F 1 "+3.3V" H 10250 4490 50  0000 C CNN
 F 2 "" H 10250 4350 60  0000 C CNN
@@
 $EndComp
 $Comp
-L GND #PWR?
+L GND #PWR027
 U 1 1 5637CFF3
 P 4200 5900
-F 0 "#PWR?" H 4200 5650 50  0001 C CNN
+F 0 "#PWR027" H 4200 5650 50  0001 C CNN
 F 1 "GND" H 4200 5750 50  0000 C CNN
 F 2 "" H 4200 5900 60  0000 C CNN
@@
 $EndComp
 $Comp
-L GND #PWR?
+L GND #PWR028
 U 1 1 5637DBF8
 P 1200 2900
-F 0 "#PWR?" H 1200 2650 50  0001 C CNN
+F 0 "#PWR028" H 1200 2650 50  0001 C CNN
 F 1 "GND" H 1200 2750 50  0000 C CNN
 F 2 "" H 1200 2900 60  0000 C CNN
@@
 Wire Wire Line
 	1350 1400 5800 1400
+Text Notes 9950 1550 0    60   ~ 0
+5V 2A
+$Comp
+L LTC3564 U?
+U 1 1 563BBE01
+P 5100 7150
+F 0 "U?" H 5100 6800 60  0000 C CNN
+F 1 "LTC3564" H 5100 7450 60  0000 C CNN
+F 2 "" H 5100 7150 60  0000 C CNN
+F 3 "" H 5100 7150 60  0000 C CNN
+	1    5100 7150
+	1    0    0    -1
+$EndComp
+Wire Wire Line
+	4050 7000 4600 7000
+Wire Wire Line
+	4600 7150 4500 7150
+Wire Wire Line
+	4500 7150 4500 7000
+Connection ~ 4500 7000
+$Comp
+L GND #PWR?
+U 1 1 563BC504
+P 4600 7600
+F 0 "#PWR?" H 4600 7350 50  0001 C CNN
+F 1 "GND" H 4600 7450 50  0000 C CNN
+F 2 "" H 4600 7600 60  0000 C CNN
+F 3 "" H 4600 7600 60  0000 C CNN
+	1    4600 7600
+	1    0    0    -1
+$EndComp
+Wire Wire Line
+	4600 7300 4600 7600
+$Comp
+L INDUCTOR L?
+U 1 1 563BC829
+P 6050 7000
+F 0 "L?" V 6000 7000 50  0000 C CNN
+F 1 "1µH" V 6150 7000 50  0000 C CNN
+F 2 "" H 6050 7000 60  0000 C CNN
+F 3 "" H 6050 7000 60  0000 C CNN
+F 4 "Vishay IHLP1616ABER1R0M01" V 6050 7000 60  0001 C CNN "Device"
+	1    6050 7000
+	0    -1   -1   0
+$EndComp
 $EndSCHEMATC

Commit message: Basic schematic with temparature and humidity sensor.
Parts:
- removed C?: 22µ, symbol C
- removed D?: ZENER, symbol ZENER
- removed L?: 1µH, symbol INDUCTOR
- removed Q? (x3): Q_PMOS_DGS, symbol Q_PMOS_DGS
- removed R? (x2): R, symbol R
- removed U?: LTC3564, symbol LTC3564
- added BT?: Battery, symbol Battery
- added D?: TVS, symbol TVS
Connections:
- wire segments 119 -> 105
Changed lines of the file:
@@
 LIBS:74xx
 LIBS:74xgxx
+LIBS:can-node
 LIBS:can-node-cache
 EELAYER 25 0
@@
 $Descr A4 11693 8268
 encoding utf-8
-Sheet 2 4
+Sheet 2 5
 Title ""
 Date ""
@@
 $EndComp
 $Comp
-L ZENER D?
-U 1 1 562BB5DB
-P -1050 -1800
-F 0 "D?" H -1050 -1700 50  0000 C CNN
-F 1 "ZENER" H -1050 -1900 50  0000 C CNN
-F 2 "" H -1050 -1800 60  0000 C CNN
-F 3 "" H -1050 -1800 60  0000 C CNN
-	1    -1050 -1800
-	0    1    1    0
-$EndComp
-$Comp
-L R R?
-U 1 1 562BC327
-P -1050 -2350
-F 0 "R?" V -970 -2350 50  0000 C CNN
-F 1 "R" V -1050 -2350 50  0000 C CNN
-F 2 "" V -1120 -2350 30  0000 C CNN
-F 3 "" H -1050 -2350 30  0000 C CNN
-	1    -1050 -2350
-	1    0    0    -1
-$EndComp
-$Comp
-L GND #PWR06
-U 1 1 562BC4C3
-P -1050 -1350
-F 0 "#PWR06" H -1050 -1600 50  0001 C CNN
-F 1 "GND" H -1050 -1500 50  0000 C CNN
-F 2 "" H -1050 -1350 60  0000 C CNN
-F 3 "" H -1050 -1350 60  0000 C CNN
-	1    -1050 -1350
-	1    0    0    -1
-$EndComp
-$Comp
-L Q_PMOS_DGS Q?
-U 1 1 562BC92C
-P -1400 -2650
-F 0 "Q?" H -1100 -2600 50  0000 R CNN
-F 1 "Q_PMOS_DGS" H -750 -2700 50  0000 R CNN
-F 2 "" H -1200 -2550 29  0000 C CNN
-F 3 "" H -1400 -2650 60  0000 C CNN
-	1    -1400 -2650
-	0    -1   -1   0
-$EndComp
-$Comp
-L Q_PMOS_DGS Q?
-U 1 1 562BCADA
-P -700 -2100
-F 0 "Q?" H -400 -2050 50  0000 R CNN
-F 1 "Q_PMOS_DGS" H -50 -2150 50  0000 R CNN
-F 2 "" H -500 -2000 29  0000 C CNN
-F 3 "" H -700 -2100 60  0000 C CNN
-	1    -700 -2100
-	1    0    0    -1
-$EndComp
-$Comp
-L Q_PMOS_DGS Q?
-U 1 1 562BCF80
-P 0 -2650
-F 0 "Q?" H 300 -2600 50  0000 R CNN
-F 1 "Q_PMOS_DGS" H 650 -2700 50  0000 R CNN
-F 2 "" H 200 -2550 29  0000 C CNN
-F 3 "" H 0   -2650 60  0000 C CNN
-	1    0    -2650
-	0    -1   -1   0
-$EndComp
-$Comp
-L R R?
-U 1 1 562BD05B
-P -200 -1600
-F 0 "R?" V -120 -1600 50  0000 C CNN
-F 1 "R" V -200 -1600 50  0000 C CNN
-F 2 "" V -270 -1600 30  0000 C CNN
-F 3 "" H -200 -1600 30  0000 C CNN
-	1    -200 -1600
-	1    0    0    -1
-$EndComp
-$Comp
-L GND #PWR07
-U 1 1 562BD4E1
-P -200 -1350
-F 0 "#PWR07" H -200 -1600 50  0001 C CNN
-F 1 "GND" H -200 -1500 50  0000 C CNN
-F 2 "" H -200 -1350 60  0000 C CNN
-F 3 "" H -200 -1350 60  0000 C CNN
-	1    -200 -1350
-	1    0    0    -1
-$EndComp
-$Comp
-L GND #PWR08
-U 1 1 562BEC1D
-P -1400 -1350
-F 0 "#PWR08" H -1400 -1600 50  0001 C CNN
-F 1 "GND" H -1400 -1500 50  0000 C CNN
-F 2 "" H -1400 -1350 60  0000 C CNN
-F 3 "" H -1400 -1350 60  0000 C CNN
-	1    -1400 -1350
-	1    0    0    -1
-$EndComp
-$Comp
 L +3.3V #PWR09
 U 1 1 562C0A20
@@
 	750  1250 750  1400
 Wire Wire Line
-	-1050 -2200 -1050 -2000
-Wire Wire Line
-	-1050 -1350 -1050 -1600
-Wire Wire Line
-	-1050 -2500 -1050 -2750
-Wire Wire Line
-	-1050 -2100 -900 -2100
-Connection ~ -1050 -2100
-Wire Wire Line
-	-600 -2300 -600 -2750
-Wire Wire Line
-	0    -1850 0    -2450
-Wire Wire Line
-	-600 -1900 -600 -1850
-Wire Wire Line
-	-600 -1850 0    -1850
-Wire Wire Line
-	-200 -1750 -200 -1850
-Connection ~ -200 -1850
-Wire Wire Line
-	-200 -1350 -200 -1450
-Wire Wire Line
-	-1400 -1350 -1400 -2450
-Wire Wire Line
 	10250 1600 10250 1400
 Wire Wire Line
@@
 Wire Wire Line
 	4950 2900 4950 2800
-$Comp
-L C C?
-U 1 1 56350ADC
-P 400 -2200
-F 0 "C?" V 300 -2100 50  0000 C CNN
-F 1 "22µ" V 550 -2200 50  0000 C CNN
-F 2 "" H 400 -2200 60  0000 C CNN
-F 3 "" H 400 -2200 60  0000 C CNN
-	1    400  -2200
-	-1   0    0    1
-$EndComp
-Wire Wire Line
-	400  -2350 400  -2750
-$Comp
-L GND #PWR015
-U 1 1 563511D1
-P 400 -1250
-F 0 "#PWR015" H 400 -1500 50  0001 C CNN
-F 1 "GND" H 400 -1400 50  0000 C CNN
-F 2 "" H 400 -1250 60  0000 C CNN
-F 3 "" H 400 -1250 60  0000 C CNN
-	1    400  -1250
-	1    0    0    -1
-$EndComp
-Wire Wire Line
-	400  -1250 400  -2050
 $Comp
 L C C?
@@
 	1600 1950 1600 2050
 Wire Wire Line
-	-1200 -2750 -200 -2750
-Wire Wire Line
 	1200 1700 1200 2300
 Wire Wire Line
@@
 5V 2A
 $Comp
-L LTC3564 U?
-U 1 1 563BBE01
-P 5100 7150
-F 0 "U?" H 5100 6800 60  0000 C CNN
-F 1 "LTC3564" H 5100 7450 60  0000 C CNN
-F 2 "" H 5100 7150 60  0000 C CNN
-F 3 "" H 5100 7150 60  0000 C CNN
-	1    5100 7150
-	1    0    0    -1
-$EndComp
-Wire Wire Line
-	4050 7000 4600 7000
-Wire Wire Line
-	4600 7150 4500 7150
-Wire Wire Line
-	4500 7150 4500 7000
-Connection ~ 4500 7000
+L Battery BT?
+U 1 1 57AF2EDA
+P 3000 6400
+F 0 "BT?" H 3118 6446 50  0000 L CNN
+F 1 "Battery" H 3118 6355 50  0000 L CNN
+F 2 "" V 3000 6440 50  0000 C CNN
+F 3 "" V 3000 6440 50  0000 C CNN
+	1    3000 6400
+	1    0    0    -1
+$EndComp
+$Comp
+L VBAT #PWR?
+U 1 1 57AF30BC
+P 3000 6000
+F 0 "#PWR?" H 3000 5850 50  0001 C CNN
+F 1 "VBAT" H 3000 6140 50  0000 C CNN
+F 2 "" H 3000 6000 60  0000 C CNN
+F 3 "" H 3000 6000 60  0000 C CNN
+	1    3000 6000
+	1    0    0    -1
+$EndComp
 $Comp
 L GND #PWR?
-U 1 1 563BC504
-P 4600 7600
-F 0 "#PWR?" H 4600 7350 50  0001 C CNN
-F 1 "GND" H 4600 7450 50  0000 C CNN
-F 2 "" H 4600 7600 60  0000 C CNN
-F 3 "" H 4600 7600 60  0000 C CNN
-	1    4600 7600
-	1    0    0    -1
-$EndComp
-Wire Wire Line
-	4600 7300 4600 7600
-$Comp
-L INDUCTOR L?
-U 1 1 563BC829
-P 6050 7000
-F 0 "L?" V 6000 7000 50  0000 C CNN
-F 1 "1µH" V 6150 7000 50  0000 C CNN
-F 2 "" H 6050 7000 60  0000 C CNN
-F 3 "" H 6050 7000 60  0000 C CNN
-F 4 "Vishay IHLP1616ABER1R0M01" V 6050 7000 60  0001 C CNN "Device"
-	1    6050 7000
-	0    -1   -1   0
-$EndComp
+U 1 1 57AF3133
+P 3000 6800
+F 0 "#PWR?" H 3000 6550 50  0001 C CNN
+F 1 "GND" H 3000 6650 50  0000 C CNN
+F 2 "" H 3000 6800 60  0000 C CNN
+F 3 "" H 3000 6800 60  0000 C CNN
+	1    3000 6800
+	1    0    0    -1
+$EndComp
+Wire Wire Line
+	3000 6000 3000 6250
+Wire Wire Line
+	3000 6550 3000 6800
+$Comp
+L TVS D?
+U 1 1 57AF3BB5
+P 850 2200
+F 0 "D?" V 804 2288 50  0000 L CNN
+F 1 "TVS" V 895 2288 50  0000 L CNN
+F 2 "" H 850 2200 50  0000 C CNN
+F 3 "" H 850 2200 50  0000 C CNN
+	1    850  2200
+	0    1    1    0
+$EndComp
+Wire Wire Line
+	850  1900 850  1400
+Connection ~ 850  1400
+$Comp
+L GND #PWR?
+U 1 1 57AF3EE9
+P 850 2900
+F 0 "#PWR?" H 850 2650 50  0001 C CNN
+F 1 "GND" H 850 2750 50  0000 C CNN
+F 2 "" H 850 2900 60  0000 C CNN
+F 3 "" H 850 2900 60  0000 C CNN
+	1    850  2900
+	1    0    0    -1
+$EndComp
+Wire Wire Line
+	850  2900 850  2500
 $EndSCHEMATC

Commit message: .
Parts:
- C10, C11, C12, C2, C3, C4, C5, C6, C7, C8, C9: renamed from C?; footprint (none) -> Capacitors_SMD:C_0603_HandSoldering
- D3: renamed from D?; footprint SOD-323 -> (none)
- Q1: renamed from Q?; footprint POWERDI3333-8 -> (none)
- R1, R10, R11, R12, R13, R14, R2, R3, R4, R5, R6, R7, R8, R9: renamed from R?; footprint (none) -> Resistors_SMD:R_0603_HandSoldering
- gave numbers to parts that had none: 10
