File: power.sch (KiCad schematic (older format))
At the start: 24 parts, among them Q1 DMP6050SFG

Commit message: Reset circuit, minor changes
Parts:
- renumbered BT1 to BT?, C1 to C?, C2 to C?, D2 to D?, D3 to D?, D1 to D?, Q1 to Q?, R2 to R?, R1 to R?
Connections:
- net labels added: PWRGD
- wire segments 69 -> 56
Changed lines of the file:
@@
 $EndDescr
 $Comp
-L CP C1
+L CP C?
 U 1 1 562B86FE
 P 1200 6700
-F 0 "C1" H 1225 6800 50  0000 L CNN
+F 0 "C?" H 1225 6800 50  0000 L CNN
 F 1 "470000uF" H 1225 6600 50  0000 L CNN
 F 2 "" H 1238 6550 30  0001 C CNN
@@
 $EndComp
 $Comp
-L R R2
+L R R?
 U 1 1 562B8880
 P 1200 6150
-F 0 "R2" V 1280 6150 50  0000 C CNN
+F 0 "R?" V 1280 6150 50  0000 C CNN
 F 1 "330" V 1200 6150 50  0000 C CNN
 F 2 "Resistors_SMD:R_0603_HandSoldering" H 1200 6150 60  0001 C CNN
@@
 $EndComp
 $Comp
-L VBAT #PWR01
+L VBAT #PWR?
 U 1 1 562B8E65
 P 2050 5450
-F 0 "#PWR01" H 2050 5300 50  0001 C CNN
+F 0 "#PWR?" H 2050 5300 50  0001 C CNN
 F 1 "VBAT" H 2050 5590 50  0000 C CNN
 F 2 "" H 2050 5450 60  0000 C CNN
@@
 $EndComp
 $Comp
-L GND #PWR02
+L GND #PWR?
 U 1 1 562B8F95
 P 1200 7000
-F 0 "#PWR02" H 1200 6750 50  0001 C CNN
+F 0 "#PWR?" H 1200 6750 50  0001 C CNN
 F 1 "GND" H 1200 6850 50  0000 C CNN
 F 2 "" H 1200 7000 60  0000 C CNN
@@
 $EndComp
 $Comp
-L C C2
+L C C?
 U 1 1 562B9539
 P 2050 6700
-F 0 "C2" V 2150 6850 50  0000 C CNN
+F 0 "C?" V 2150 6850 50  0000 C CNN
 F 1 "100n" V 2150 6550 50  0000 C CNN
 F 2 "Capacitors_SMD:C_0603_HandSoldering" H 2050 6700 60  0001 C CNN
@@
 $EndComp
 $Comp
-L GND #PWR03
+L GND #PWR?
 U 1 1 562B96C2
 P 2050 7000
-F 0 "#PWR03" H 2050 6750 50  0001 C CNN
+F 0 "#PWR?" H 2050 6750 50  0001 C CNN
 F 1 "GND" H 2050 6850 50  0000 C CNN
 F 2 "" H 2050 7000 60  0000 C CNN
@@
 $EndComp
 $Comp
-L VIN #PWR05
+L VIN #PWR?
 U 1 1 562BB258
 P 750 1250
-F 0 "#PWR05" H 750 1100 50  0001 C CNN
+F 0 "#PWR?" H 750 1100 50  0001 C CNN
 F 1 "VIN" H 750 1390 50  0000 C CNN
 F 2 "" H 750 1250 60  0000 C CNN
@@
 $EndComp
 $Comp
-L +3.3V #PWR06
+L +3.3V #PWR?
 U 1 1 562C0A20
 P 1200 5450
-F 0 "#PWR06" H 1200 5300 50  0001 C CNN
+F 0 "#PWR?" H 1200 5300 50  0001 C CNN
 F 1 "+3.3V" H 1200 5590 50  0000 C CNN
 F 2 "" H 1200 5450 60  0000 C CNN
@@
 $EndComp
 $Comp
-L D D2
+L D D?
 U 1 1 562B8819
 P 1200 5750
-F 0 "D2" H 1200 5850 50  0000 C CNN
+F 0 "D?" H 1200 5850 50  0000 C CNN
 F 1 "D" H 1200 5650 50  0000 C CNN
 F 2 "" H 1200 5750 60  0001 C CNN
@@
 12..24 V
 $Comp
-L R R1
+L R R?
 U 1 1 5637DBF2
 P 1200 2450
-F 0 "R1" V 1280 2450 50  0000 C CNN
+F 0 "R?" V 1280 2450 50  0000 C CNN
 F 1 "100k" V 1200 2450 50  0000 C CNN
 F 2 "Resistors_SMD:R_0603_HandSoldering" V 1130 2450 30  0001 C CNN
@@
 $EndComp
 $Comp
-L GND #PWR024
+L GND #PWR?
 U 1 1 5637DBF8
 P 1200 2900
-F 0 "#PWR024" H 1200 2650 50  0001 C CNN
+F 0 "#PWR?" H 1200 2650 50  0001 C CNN
 F 1 "GND" H 1200 2750 50  0000 C CNN
 F 2 "" H 1200 2900 60  0000 C CNN
@@
 $EndComp
 $Comp
-L ZENER D3
+L ZENER D?
 U 1 1 5637E04D
 P 1600 1750
-F 0 "D3" H 1600 1850 50  0000 C CNN
+F 0 "D?" H 1600 1850 50  0000 C CNN
 F 1 "10V" H 1600 1650 50  0000 C CNN
 F 2 "" H 1600 1750 60  0001 C CNN
@@
 $EndComp
 $Comp
-L DMP6050SFG Q1
+L DMP6050SFG Q?
 U 1 1 563833E4
 P 1150 1450
-F 0 "Q1" H 1300 1550 50  0000 L CNN
+F 0 "Q?" H 1300 1550 50  0000 L CNN
 F 1 "DMP6050SFG" H 1300 1450 50  0000 L CNN
 F 2 "" H 1300 1350 50  0001 L CNN
@@
 $EndComp
 $Comp
-L Battery BT1
+L Battery BT?
 U 1 1 57AF2EDA
 P 2650 6400
-F 0 "BT1" H 2768 6446 50  0000 L CNN
+F 0 "BT?" H 2768 6446 50  0000 L CNN
 F 1 "Battery" H 2768 6355 50  0000 L CNN
 F 2 "" V 2650 6440 50  0001 C CNN
@@
 $EndComp
 $Comp
-L VBAT #PWR025
+L VBAT #PWR?
 U 1 1 57AF30BC
 P 2650 6000
-F 0 "#PWR025" H 2650 5850 50  0001 C CNN
+F 0 "#PWR?" H 2650 5850 50  0001 C CNN
 F 1 "VBAT" H 2650 6140 50  0000 C CNN
 F 2 "" H 2650 6000 60  0000 C CNN
@@
 $EndComp
 $Comp
-L GND #PWR026
+L GND #PWR?
 U 1 1 57AF3133
 P 2650 6800
-F 0 "#PWR026" H 2650 6550 50  0001 C CNN
+F 0 "#PWR?" H 2650 6550 50  0001 C CNN
 F 1 "GND" H 2650 6650 50  0000 C CNN
 F 2 "" H 2650 6800 60  0000 C CNN
@@
 $EndComp
 $Comp
-L TVS D1
+L TVS D?
 U 1 1 57AF3BB5
 P 850 2200
-F 0 "D1" V 804 2288 50  0000 L CNN
+F 0 "D?" V 804 2288 50  0000 L CNN
 F 1 "TVS" V 895 2288 50  0000 L CNN
 F 2 "" H 850 2200 50  0001 C CNN
@@
 $EndComp
 $Comp
-L GND #PWR027
+L GND #PWR?
 U 1 1 57AF3EE9
 P 850 2900
-F 0 "#PWR027" H 850 2650 50  0001 C CNN
+F 0 "#PWR?" H 850 2650 50  0001 C CNN
 F 1 "GND" H 850 2750 50  0000 C CNN
 F 2 "" H 850 2900 60  0000 C CNN
@@
 	1200 5900 1200 6000
 Wire Wire Line
-	1200 6300 1200 6400
-Wire Wire Line
-	1200 6400 1200 6550
+	1200 6300 1200 6550
 Wire Wire Line
 	1200 6850 1200 7000
@@
 	1200 6400 2050 6400
 Wire Wire Line
-	2050 5450 2050 6400
-Wire Wire Line
-	2050 6400 2050 6550
+	2050 5450 2050 6550
 Connection ~ 1200 6400
 Connection ~ 2050 6400
@@
 	1600 1950 1600 2050
 Wire Wire Line
-	1200 1700 1200 2050
-Wire Wire Line
-	1200 2050 1200 2300
+	1200 1700 1200 2300
 Wire Wire Line
 	1600 2050 1200 2050
@@
 Connection ~ 1600 1400
 Wire Wire Line
-	750  1400 850  1400
-Wire Wire Line
-	850  1400 950  1400
+	750  1400 950  1400
 Wire Wire Line
 	2650 6000 2650 6250
@@
 $EndComp
 Wire Wire Line
-	1350 1400 1600 1400
-Wire Wire Line
-	1600 1400 3100 1400
-Wire Wire Line
-	3100 1400 3450 1400
-Wire Wire Line
-	3450 1400 4700 1400
+	1350 1400 4700 1400
 Wire Wire Line
 	3450 1500 3450 1400
 Connection ~ 3450 1400
 Wire Wire Line
-	3450 1800 3450 1850
-Wire Wire Line
-	3450 1850 3450 2000
+	3450 1800 3450 2000
 Wire Wire Line
 	3450 2300 3450 2450
@@
 	4600 2750 4600 2950
 Wire Wire Line
-	4350 2300 4600 2300
-Wire Wire Line
-	4600 2300 4700 2300
+	4350 2300 4700 2300
 Wire Wire Line
 	4350 2300 4350 2650
@@
 Connection ~ 4600 2300
 Wire Wire Line
-	5900 1900 6450 1900
-Wire Wire Line
-	6450 1900 6700 1900
-Wire Wire Line
-	6450 1700 6450 1900
-Wire Wire Line
-	6450 1900 6450 2000
+	5900 1900 6700 1900
+Wire Wire Line
+	6450 1700 6450 2000
 Connection ~ 6450 1900
 Wire Wire Line
-	7300 1900 7400 1900
-Wire Wire Line
-	7400 1900 7850 1900
-Wire Wire Line
-	7850 1900 8450 1900
+	7300 1900 8450 1900
 Wire Wire Line
 	7400 2000 7400 1900
 Connection ~ 7400 1900
 Wire Wire Line
-	7400 2300 7400 2600
-Wire Wire Line
-	7400 2600 7400 2650
+	7400 2300 7400 2650
 Wire Wire Line
 	5900 2200 5900 2600
@@
 Wire Wire Line
 	8450 1900 8450 1700
+Text GLabel 6600 1400 2    60   Output ~ 0
+PWRGD
+Wire Wire Line
+	6600 1400 5900 1400
 $EndSCHEMATC

Commit message: .
Parts:
- removed C?: 470000uF, symbol CP
- removed C?: 100n, Capacitors_SMD:C_0603_HandSoldering, symbol C
- removed D?: D, symbol D
- removed R?: 330, Resistors_SMD:R_0603_HandSoldering, symbol R
- BT1: renamed from BT?; footprint (none) -> Battery_Holders:Keystone_106_1x20mm-CoinCell
- C4, C6, C7: renamed from C?; footprint (none) -> Capacitors_SMD:C_0603
- R1: renamed from R?; footprint Resistors_SMD:R_0603_HandSoldering -> Resistors_SMD:R_0603
- U1: renamed from U?; footprint (none) -> can-node:TI-DGQ
- gave numbers to parts that had none: 14
Connections:
- net labels added: +3.3VADC, GNDA
- wire segments 56 -> 53

Commit message: 24 V input protection
Parts:
- removed Q1: DMP6050SFG, symbol DMP6050SFG
- added Q1: DMP6023LSS, Power_Integrations:SO-8, symbol DMP6023LSS
- D1: value TVS -> 40.2V; Part (none) -> P4SMA47CA
- renumbered C3 to C1, C4 to C2, C5 to C3, C6 to C4, C7 to C5, C8 to C6, D3 to D2, D4 to D3, R3 to R2, R4 to R3, R5 to R4, R6 to R5, R7 to R6, R8 to R7
Changed lines of the file:
@@
 $EndComp
 $Comp
-L ZENER D3
+L ZENER D2
 U 1 1 5637E04D
 P 1600 1750
-F 0 "D3" H 1600 1850 50  0000 C CNN
+F 0 "D2" H 1600 1850 50  0000 C CNN
 F 1 "10V" H 1600 1650 50  0000 C CNN
 F 2 "" H 1600 1750 60  0001 C CNN
@@
 	1    1600 1750
 	0    1    1    0
-$EndComp
-$Comp
-L DMP6050SFG Q1
-U 1 1 563833E4
-P 1150 1450
-F 0 "Q1" H 1300 1550 50  0000 L CNN
-F 1 "DMP6050SFG" H 1300 1450 50  0000 L CNN
-F 2 "" H 1300 1350 50  0001 L CNN
-F 3 "" H 1100 1450 50  0000 L CNN
-	1    1150 1450
-	0    -1   -1   0
 $EndComp
 $Comp
@@
 P 850 2200
 F 0 "D1" V 804 2288 50  0000 L CNN
-F 1 "TVS" V 895 2288 50  0000 L CNN
+F 1 "40.2V" V 895 2288 50  0000 L CNN
 F 2 "" H 850 2200 50  0001 C CNN
-F 3 "" H 850 2200 50  0000 C CNN
+F 3 "http://www.vishay.com/docs/88367/p4sma.pdf" H 850 2200 50  0001 C CNN
+F 4 "P4SMA47CA" V 1100 2200 60  0000 C CNN "Part"
 	1    850  2200
 	0    1    1    0
@@
 $EndComp
 $Comp
-L R R3
+L R R2
 U 1 1 57B90F3D
 P 3450 1650
-F 0 "R3" H 3520 1696 50  0000 L CNN
+F 0 "R2" H 3520 1696 50  0000 L CNN
 F 1 "105k" H 3520 1605 50  0000 L CNN
 F 2 "" V 3380 1650 50  0001 C CNN
@@
 $EndComp
 $Comp
-L R R4
+L R R3
 U 1 1 57B90F43
 P 3450 2150
-F 0 "R4" H 3520 2196 50  0000 L CNN
+F 0 "R3" H 3520 2196 50  0000 L CNN
 F 1 "16k9" H 3520 2105 50  0000 L CNN
 F 2 "" V 3380 2150 50  0001 C CNN
@@
 $EndComp
 $Comp
-L C C3
+L C C1
 U 1 1 57B90F4F
 P 3100 1950
-F 0 "C3" H 3215 1996 50  0000 L CNN
+F 0 "C1" H 3215 1996 50  0000 L CNN
 F 1 "2µ2" H 3215 1905 50  0000 L CNN
 F 2 "" H 3138 1800 50  0001 C CNN
@@
 $EndComp
 $Comp
-L C C5
+L C C3
 U 1 1 57B90F5C
 P 4350 2800
-F 0 "C5" H 4465 2846 50  0000 L CNN
+F 0 "C3" H 4465 2846 50  0000 L CNN
 F 1 "1p3" H 4465 2755 50  0000 L CNN
 F 2 "" H 4388 2650 50  0001 C CNN
@@
 $EndComp
 $Comp
-L C C6
+L C C4
 U 1 1 57B90F62
 P 4600 3100
-F 0 "C6" H 4715 3146 50  0000 L CNN
+F 0 "C4" H 4715 3146 50  0000 L CNN
 F 1 "1n8" H 4715 3055 50  0000 L CNN
 F 2 "Capacitors_SMD:C_0603" H 4638 2950 50  0001 C CNN
@@
 $EndComp
 $Comp
-L C C4
+L C C2
 U 1 1 57B90F68
 P 3800 3150
-F 0 "C4" H 3915 3196 50  0000 L CNN
+F 0 "C2" H 3915 3196 50  0000 L CNN
 F 1 "6n8" H 3915 3105 50  0000 L CNN
 F 2 "Capacitors_SMD:C_0603" H 3838 3000 50  0001 C CNN
@@
 $EndComp
 $Comp
-L R R6
+L R R5
 U 1 1 57B90F6E
 P 4600 2600
-F 0 "R6" H 4670 2646 50  0000 L CNN
+F 0 "R5" H 4670 2646 50  0000 L CNN
 F 1 "147k" H 4670 2555 50  0000 L CNN
 F 2 "" V 4530 2600 50  0001 C CNN
@@
 $EndComp
 $Comp
-L R R5
+L R R4
 U 1 1 57B90F7A
 P 4050 2850
-F 0 "R5" H 4120 2896 50  0000 L CNN
+F 0 "R4" H 4120 2896 50  0000 L CNN
 F 1 "309k" H 4120 2805 50  0000 L CNN
 F 2 "" V 3980 2850 50  0001 C CNN
@@
 $EndComp
 $Comp
-L R R7
+L R R6
 U 1 1 57B90F92
 P 7400 2150
-F 0 "R7" H 7470 2196 50  0000 L CNN
+F 0 "R6" H 7470 2196 50  0000 L CNN
 F 1 "31k6" H 7470 2105 50  0000 L CNN
 F 2 "" V 7330 2150 50  0001 C CNN
@@
 $EndComp
 $Comp
-L C C7
+L C C5
 U 1 1 57B90F99
 P 6150 1700
-F 0 "C7" V 5898 1700 50  0000 C CNN
+F 0 "C5" V 5898 1700 50  0000 C CNN
 F 1 "100n" V 5989 1700 50  0000 C CNN
 F 2 "Capacitors_SMD:C_0603" H 6188 1550 50  0001 C CNN
@@
 $EndComp
 $Comp
-L D_Schottky D4
+L D_Schottky D3
 U 1 1 57B90F9F
 P 6450 2150
-F 0 "D4" V 6404 2229 50  0000 L CNN
+F 0 "D3" V 6404 2229 50  0000 L CNN
 F 1 "0.51V 0.5A" V 6495 2229 50  0000 L CNN
 F 2 "" H 6450 2150 50  0001 C CNN
@@
 $EndComp
 $Comp
-L R R8
+L R R7
 U 1 1 57B90FAB
 P 7400 2800
-F 0 "R8" H 7470 2846 50  0000 L CNN
+F 0 "R7" H 7470 2846 50  0000 L CNN
 F 1 "10k" H 7470 2755 50  0000 L CNN
 F 2 "" V 7330 2800 50  0001 C CNN
@@
 	5200 2700 5200 2800
 $Comp
-L C C8
+L C C6
 U 1 1 57B90FFB
 P 7850 2400
-F 0 "C8" H 7965 2446 50  0000 L CNN
+F 0 "C6" H 7965 2446 50  0000 L CNN
 F 1 "47µ" H 7965 2355 50  0000 L CNN
 F 2 "" H 7888 2250 50  0001 C CNN
@@
 Wire Wire Line
 	4700 5450 4700 5400
+$Comp
+L DMP6023LSS Q1
+U 1 1 57C95065
+P 1150 1500
+F 0 "Q1" V 1450 1500 50  0000 C CNN
+F 1 "DMP6023LSS" V 1350 1500 50  0000 C CNN
+F 2 "Power_Integrations:SO-8" V 1100 1750 50  0001 C CIN
+F 3 "" H 1150 1500 50  0000 L CNN
+	1    1150 1500
+	0    1    -1   0
+$EndComp
 $EndSCHEMATC

Commit message: Add bom, minor changes
Parts:
- BT1: footprint Battery_Holders:Keystone_106_1x20mm-CoinCell -> (none)
- C1: footprint (none) -> Capacitors_SMD:C_1206
- C2, C4, C5: footprint Capacitors_SMD:C_0603 -> (none)
- D1: footprint (none) -> can-node:DO-214AC
- D2: footprint (none) -> Diodes_SMD:SMA_Standard; Device ON Semiconductor MM3Z10VT1G -> ON Semiconductor 1SMA5925BT3G
- L1: value 56µF, 0.24Ω -> 56µH 0.24Ω
- Q1: footprint Power_Integrations:SO-8 -> can-node:DMP6023LSS
- R1: footprint Resistors_SMD:R_0603 -> Resistors_SMD:R_1206
- R2, R3, R4, R5, R6, R7: footprint (none) -> Resistors_SMD:R_0603
- U1: footprint can-node:TI-DGQ -> (none)
Changed lines of the file:
@@
 F 0 "R1" V 1280 2450 50  0000 C CNN
 F 1 "100k" V 1200 2450 50  0000 C CNN
-F 2 "Resistors_SMD:R_0603" V 1130 2450 30  0001 C CNN
+F 2 "Resistors_SMD:R_1206" V 1130 2450 30  0001 C CNN
 F 3 "" H 1200 2450 30  0000 C CNN
 	1    1200 2450
@@
 F 0 "D2" H 1600 1850 50  0000 C CNN
 F 1 "10V" H 1600 1650 50  0000 C CNN
-F 2 "" H 1600 1750 60  0001 C CNN
+F 2 "Diodes_SMD:SMA_Standard" H 1600 1750 60  0001 C CNN
 F 3 "http://www.onsemi.com/pub_link/Collateral/MM3Z2V4T1-D.PDF" H 1600 1750 60  0001 C CNN
-F 4 "ON Semiconductor MM3Z10VT1G" H 1600 1750 60  0001 C CNN "Device"
+F 4 "ON Semiconductor 1SMA5925BT3G" H 1600 1750 60  0001 C CNN "Device"
 	1    1600 1750
 	0    1    1    0
@@
 F 0 "BT1" H 2768 6446 50  0000 L CNN
 F 1 "Battery" H 2768 6355 50  0000 L CNN
-F 2 "Battery_Holders:Keystone_106_1x20mm-CoinCell" V 2650 6440 50  0001 C CNN
+F 2 "" V 2650 6440 50  0001 C CNN
 F 3 "" V 2650 6440 50  0000 C CNN
 	1    2650 6400
@@
 F 0 "D1" V 804 2288 50  0000 L CNN
 F 1 "40.2V" V 895 2288 50  0000 L CNN
-F 2 "" H 850 2200 50  0001 C CNN
+F 2 "can-node:DO-214AC" H 850 2200 50  0001 C CNN
 F 3 "http://www.vishay.com/docs/88367/p4sma.pdf" H 850 2200 50  0001 C CNN
 F 4 "P4SMA47CA" V 1100 2200 60  0000 C CNN "Part"
@@
 F 0 "U1" H 5300 2687 60  0000 C CNN
 F 1 "TPS5401" H 5300 2581 60  0000 C CNB
-F 2 "can-node:TI-DGQ" H 5300 1900 60  0001 C CNN
+F 2 "" H 5300 1900 60  0001 C CNN
 F 3 "" H 5300 1900 60  0000 C CNN
 	1    5300 1900
@@
 F 0 "R2" H 3520 1696 50  0000 L CNN
 F 1 "105k" H 3520 1605 50  0000 L CNN
-F 2 "" V 3380 1650 50  0001 C CNN
+F 2 "Resistors_SMD:R_0603" V 3380 1650 50  0001 C CNN
 F 3 "" H 3450 1650 50  0000 C CNN
 	1    3450 1650
@@
 F 0 "R3" H 3520 2196 50  0000 L CNN
 F 1 "16k9" H 3520 2105 50  0000 L CNN
-F 2 "" V 3380 2150 50  0001 C CNN
+F 2 "Resistors_SMD:R_0603" V 3380 2150 50  0001 C CNN
 F 3 "" H 3450 2150 50  0000 C CNN
 	1    3450 2150
@@
 F 0 "C1" H 3215 1996 50  0000 L CNN
 F 1 "2µ2" H 3215 1905 50  0000 L CNN
-F 2 "" H 3138 1800 50  0001 C CNN
+F 2 "Capacitors_SMD:C_1206" H 3138 1800 50  0001 C CNN
 F 3 "" H 3100 1950 50  0000 C CNN
 	1    3100 1950
@@
 F 0 "C4" H 4715 3146 50  0000 L CNN
 F 1 "1n8" H 4715 3055 50  0000 L CNN
-F 2 "Capacitors_SMD:C_0603" H 4638 2950 50  0001 C CNN
+F 2 "" H 4638 2950 50  0001 C CNN
 F 3 "" H 4600 3100 50  0000 C CNN
 	1    4600 3100
@@
 F 0 "C2" H 3915 3196 50  0000 L CNN
 F 1 "6n8" H 3915 3105 50  0000 L CNN
-F 2 "Capacitors_SMD:C_0603" H 3838 3000 50  0001 C CNN
+F 2 "" H 3838 3000 50  0001 C CNN
 F 3 "" H 3800 3150 50  0000 C CNN
 	1    3800 3150
@@
 F 0 "R5" H 4670 2646 50  0000 L CNN
 F 1 "147k" H 4670 2555 50  0000 L CNN
-F 2 "" V 4530 2600 50  0001 C CNN
+F 2 "Resistors_SMD:R_0603" V 4530 2600 50  0001 C CNN
 F 3 "" H 4600 2600 50  0000 C CNN
 	1    4600 2600
@@
 F 0 "R4" H 4120 2896 50  0000 L CNN
 F 1 "309k" H 4120 2805 50  0000 L CNN
-F 2 "" V 3980 2850 50  0001 C CNN
+F 2 "Resistors_SMD:R_0603" V 3980 2850 50  0001 C CNN
 F 3 "" H 4050 2850 50  0000 C CNN
 	1    4050 2850
@@
 F 0 "R6" H 7470 2196 50  0000 L CNN
 F 1 "31k6" H 7470 2105 50  0000 L CNN
-F 2 "" V 7330 2150 50  0001 C CNN
+F 2 "Resistors_SMD:R_0603" V 7330 2150 50  0001 C CNN
 F 3 "" H 7400 2150 50  0000 C CNN
 	1    7400 2150
@@
 F 0 "C5" V 5898 1700 50  0000 C CNN
 F 1 "100n" V 5989 1700 50  0000 C CNN
-F 2 "Capacitors_SMD:C_0603" H 6188 1550 50  0001 C CNN
+F 2 "" H 6188 1550 50  0001 C CNN
 F 3 "" H 6150 1700 50  0000 C CNN
 F 4 "10V" V 6150 1700 60  0001 C CNN "Rating"
@@
 P 7000 1900
 F 0 "L1" V 7216 1900 50  0000 C CNN
-F 1 "56µF, 0.24Ω" V 7125 1900 50  0000 C CNN
+F 1 "56µH 0.24Ω" V 7125 1900 50  0000 C CNN
 F 2 "" H 7000 1900 50  0001 C CNN
 F 3 "" H 7000 1900 50  0000 C CNN
@@
 F 0 "R7" H 7470 2846 50  0000 L CNN
 F 1 "10k" H 7470 2755 50  0000 L CNN
-F 2 "" V 7330 2800 50  0001 C CNN
+F 2 "Resistors_SMD:R_0603" V 7330 2800 50  0001 C CNN
 F 3 "" H 7400 2800 50  0000 C CNN
 	1    7400 2800
@@
 F 0 "Q1" V 1450 1500 50  0000 C CNN
 F 1 "DMP6023LSS" V 1350 1500 50  0000 C CNN
-F 2 "Power_Integrations:SO-8" V 1100 1750 50  0001 C CIN
+F 2 "can-node:DMP6023LSS" V 1100 1750 50  0001 C CIN
 F 3 "" H 1150 1500 50  0000 L CNN
 	1    1150 1500

Commit message: Bom work
Parts:
- C2: footprint (none) -> Capacitors_SMD:C_0805
- C3: value 1p3 -> 1.3p; footprint (none) -> Capacitors_SMD:C_0402
- C4: value 1n8 -> 1.8n; footprint (none) -> Capacitors_SMD:C_0402
- C5: value 100n -> 100n 10V; footprint (none) -> Capacitors_SMD:C_0402
- C6: footprint (none) -> Capacitors_SMD:C_1206
- D3: value 0.51V 0.5A -> 0.7V 1A; footprint (none) -> Diodes_SMD:SMA_Standard
Changed lines of the file:
@@
 P 4350 2800
 F 0 "C3" H 4465 2846 50  0000 L CNN
-F 1 "1p3" H 4465 2755 50  0000 L CNN
-F 2 "" H 4388 2650 50  0001 C CNN
+F 1 "1.3p" H 4465 2755 50  0000 L CNN
+F 2 "Capacitors_SMD:C_0402" H 4388 2650 50  0001 C CNN
 F 3 "" H 4350 2800 50  0000 C CNN
 F 4 "50V" H 4350 2800 60  0001 C CNN "Rating"
@@
 P 4600 3100
 F 0 "C4" H 4715 3146 50  0000 L CNN
-F 1 "1n8" H 4715 3055 50  0000 L CNN
-F 2 "" H 4638 2950 50  0001 C CNN
+F 1 "1.8n" H 4715 3055 50  0000 L CNN
+F 2 "Capacitors_SMD:C_0402" H 4638 2950 50  0001 C CNN
 F 3 "" H 4600 3100 50  0000 C CNN
 	1    4600 3100
@@
 F 0 "C2" H 3915 3196 50  0000 L CNN
 F 1 "6n8" H 3915 3105 50  0000 L CNN
-F 2 "" H 3838 3000 50  0001 C CNN
+F 2 "Capacitors_SMD:C_0805" H 3838 3000 50  0001 C CNN
 F 3 "" H 3800 3150 50  0000 C CNN
 	1    3800 3150
@@
 P 6150 1700
 F 0 "C5" V 5898 1700 50  0000 C CNN
-F 1 "100n" V 5989 1700 50  0000 C CNN
-F 2 "" H 6188 1550 50  0001 C CNN
+F 1 "100n 10V" V 5989 1700 50  0000 C CNN
+F 2 "Capacitors_SMD:C_0402" H 6188 1550 50  0001 C CNN
 F 3 "" H 6150 1700 50  0000 C CNN
 F 4 "10V" V 6150 1700 60  0001 C CNN "Rating"
@@
 P 6450 2150
 F 0 "D3" V 6404 2229 50  0000 L CNN
-F 1 "0.51V 0.5A" V 6495 2229 50  0000 L CNN
-F 2 "" H 6450 2150 50  0001 C CNN
+F 1 "0.7V 1A" V 6495 2229 50  0000 L CNN
+F 2 "Diodes_SMD:SMA_Standard" H 6450 2150 50  0001 C CNN
 F 3 "" H 6450 2150 50  0000 C CNN
 	1    6450 2150
@@
 F 0 "C6" H 7965 2446 50  0000 L CNN
 F 1 "47µ" H 7965 2355 50  0000 L CNN
-F 2 "" H 7888 2250 50  0001 C CNN
+F 2 "Capacitors_SMD:C_1206" H 7888 2250 50  0001 C CNN
 F 3 "" H 7850 2400 50  0000 C CNN
 	1    7850 2400

Commit message: Use LMR16006 DCDC
Parts:
- added C?: 100n 10V, Capacitors_SMD:C_0402, symbol C
- added C? (x2): C, symbol C
- added D?: D_Schottky, symbol D_Schottky
- added L?: INDUCTOR, symbol INDUCTOR
- added R? (x2): R, symbol R
- added R?: 100k, symbol R
- added U?: LMR16006, symbol LMR16006
- renumbered BT1 to BT?, C1 to C?, C3 to C?, C4 to C?, C2 to C?, C5 to C?, C6 to C?, D2 to D?, D1 to D?, D3 to D?, L1 to L?, Q1 to Q?, R1 to R?, R2 to R?, R3 to R?, R5 to R?, R4 to R?, R6 to R?, R7 to R?, U1 to U?
Connections:
- net +3.3VADC: now also C?.1, L?.2, R?.1
- net GND: now also C?.2, C?.2, D?.2 (A), R?.2, U?.2 (GND)
- net at C?.1, R?.1, U?.2 (VIN): no longer D?.1 (K), Q?.1 (S)
- net +5V: no longer names the net of C?.1, L?.2, R?.1
- new net: C?.1, D?.1 (K), Q?.1 (S), R?.1, U?.5 (VIN)
- new net: C?.2, U?.1 (CB)
- new net: R?.1, R?.2, U?.3 (FB)
- new net: R?.2, U?.4 (~SHDN)
- new net: C?.1, D?.1 (K), L?.1, U?.6 (SW)
Other:
- note added: "3.3V 0.6A"
- moved on the sheet: C?, D?, L?, R?, U?

Commit message: Power supply work
Parts:
- removed C?: 2µ2, Capacitors_SMD:C_1206, symbol C
- removed C?: 1.3p, Capacitors_SMD:C_0402, symbol C
- removed C?: 1.8n, Capacitors_SMD:C_0402, symbol C
- removed C?: 6n8, Capacitors_SMD:C_0805, symbol C
- removed C?: 100n 10V, Capacitors_SMD:C_0402, symbol C
- removed C?: 47µ, Capacitors_SMD:C_1206, symbol C
- removed D?: 0.7V 1A, Diodes_SMD:SMA_Standard, symbol D_Schottky
- removed L?: 56µH 0.24Ω, symbol INDUCTOR
- removed R?: 105k, Resistors_SMD:R_0603, symbol R
- removed R?: 16k9, Resistors_SMD:R_0603, symbol R
- removed R?: 147k, Resistors_SMD:R_0603, symbol R
- removed R?: 309k, Resistors_SMD:R_0603, symbol R
- removed R?: 31k6, Resistors_SMD:R_0603, symbol R
- removed R?: 10k, Resistors_SMD:R_0603, symbol R
- removed U?: TPS5401, symbol TPS5401
- C?: value C -> 22µF
- C?: value C -> 2.2µF
- D?: value D_Schottky -> 0.57V 1A
- L?: value INDUCTOR -> 27µH 220mΩ
- R?: value R -> 28k
- R?: value R -> 8.45k
Other:
- note added: "24 V"
- note removed: "12..24 V"
- note removed: "3.3V 0.5A"
- moved on the sheet: C?

Commit message: Remove power good logic
Changed lines of the file:
@@
 	1600 1950 1600 2050
 Wire Wire Line
-	1200 1700 1200 2050
-Wire Wire Line
-	1200 2050 1200 2300
+	1200 1700 1200 2300
 Wire Wire Line
 	1600 2050 1200 2050
@@
 Connection ~ 1600 1400
 Wire Wire Line
-	750  1400 850  1400
-Wire Wire Line
-	850  1400 950  1400
+	750  1400 950  1400
 Wire Wire Line
 	2650 6000 2650 6250
@@
 	850  2900 850  2500
 Wire Wire Line
-	1350 1400 1600 1400
-Wire Wire Line
-	1600 1400 2350 1400
-Wire Wire Line
-	2350 1400 2750 1400
-Wire Wire Line
-	2750 1400 2900 1400
+	1350 1400 2900 1400
 $Comp
 L GND #PWR?
@@
 	4100 1400 4150 1400
 Wire Wire Line
-	4150 1400 4150 1600
-Wire Wire Line
-	4150 1600 4150 1650
-Wire Wire Line
-	3700 1600 4150 1600
-Wire Wire Line
-	4150 1600 4250 1600
+	4150 1400 4150 1650
+Wire Wire Line
+	3700 1600 4250 1600
 $Comp
 L GND #PWR?
@@
 	2350 1800 2350 1850
 Wire Wire Line
-	4850 1600 4950 1600
-Wire Wire Line
-	4950 1600 5350 1600
-Wire Wire Line
-	5350 1600 5950 1600
+	4850 1600 5950 1600
 Wire Wire Line
 	4950 1600 4950 1650
 Wire Wire Line
-	4950 1950 4950 2000
-Wire Wire Line
-	4950 2000 4950 2050
+	4950 1950 4950 2050
 Wire Wire Line
 	4950 2400 4950 2350
