File: microcontroller.sch (KiCad schematic (older format))
At the start: 17 parts, among them P1 DEBUG_UART, P2 SWD, SW1 SW_PUSH, U3 STM32F072RB, U4 HDC1080, X1 32.768KHz 10p

Commit message: Reset circuit, minor changes
Parts:
- removed Q?: Q_NMOS_DGS, symbol Q_NMOS_DGS
- added C? (x3): 100n, symbol C
- added C? (x2): 100n, Capacitors_SMD:C_0603_HandSoldering, symbol C
- added C? (x2): 4µ7, symbol C
- added R? (x2): 10k, Resistors_SMD:R_0603_HandSoldering, symbol R
- added R? (x2): 220, Resistors_SMD:R_0603_HandSoldering, symbol R
- added SW? (x2): SW_PUSH, symbol SW_PUSH
- added U?: SN74LVC1G11, symbol SN74LVC1G11
- renumbered C18 to C?, C15 to C?, C21 to C?, C20 to C?, C19 to C?, C17 to C?, C16 to C?, C22 to C?, P1 to P?, P2 to P?, R15 to R?, R16 to R?, SW1 to SW?, U3 to U?, U4 to U?, X1 to X?
Connections:
- net +3V3: now also U?.13 (VDDA), U?.48 (VDDIO2), C?.1, C?.1, C?.1, C?.1, C?.1, R?.1, R?.1, U?.5 (VCC)
- net GND: now also SW?.2, C?.2, C?.2, C?.2, C?.2, C?.2, C?.2, C?.2, SW?.1, SW?.1, U?.2 (GND); no longer SW?.1
- net at U?.52 (PC11): now also C?.1, R?.2
- net at U?.53 (PC12): now also C?.1, R?.2
- net at C?.1, U?.7 (NRST): now also U?.4 (Y); no longer P?.4 (P4), SW?.2
- new net: R?.2, SW?.1, U?.3 (B)
- new net: P?.4 (P4), U?.6 (C)
- new net: R?.1, SW?.2 (x2)
- new net PWRGD: R?.2, U?.1 (A)
Other:
- moved on the sheet: C?, P?, SW?

Commit message: .
Parts:
- added D5, D6: red, LEDs:LED_0603, symbol Led_Small
- added R11, R12: 220, Resistors_SMD:R_0603, symbol R
- C10, C12, C14, C20, C22, C9: renamed from C?; footprint (none) -> Capacitors_SMD:C_0603
- C13, C16, C17, C18, C19: renamed from C?; footprint Capacitors_SMD:C_0603_HandSoldering -> Capacitors_SMD:C_0603
- C23: renamed from C?; value C -> 100n; footprint (none) -> Capacitors_SMD:C_0603
- R10, R13, R14, R15, R16, R9: renamed from R?; footprint Resistors_SMD:R_0603_HandSoldering -> Resistors_SMD:R_0603
- U4: renamed from U?; footprint (none) -> can-node:TI-DMB
- gave numbers to parts that had none: 11
Connections:
- net +3V3: no longer C11.1, C13.1, U3.13 (VDDA)
- net GND: now also R11.1, R12.1; no longer C11.2, C13.2, U3.12 (VSSA)
- net at U3.26 (PB0): now also D5.2 (A)
- net at U3.27 (PB1): now also D6.2 (A)
- new net: D6.1 (K), R12.2
- new net: D5.1 (K), R11.2
- new net +3.3VADC: C11.1, C13.1, U3.13 (VDDA)
- new net GNDA: C11.2, C13.2, U3.12 (VSSA)
Other:
- moved on the sheet: R16
