File: microcontroller.sch (KiCad schematic (older format))
At the start: 34 parts, among them P1 SWD, P2 DEBUG_UART, SW1 SW_PUSH, SW2 SW_PUSH, SW3 SW_PUSH, U2 SN74LVC1G08, U3 STM32F072RB, U4 HDC1080, X1 32.768KHz 12.5pF

Commit message: Layout: first version
Parts:
- added D6: LED_RGB_EP, CAN_Node:Everlight_19-337, symbol LED_RGB_6P
- added P4, P5: CONN_01X08, Pin_Headers:Pin_Header_Straight_1x08, symbol CONN_01X08
- added R15, R16, R17: 220, Resistors_SMD:R_0402, symbol R
Connections:
- net labels added: PB0, PB1, PB2, PB3, PB4, PB5, PB6, PB7, PC0, PC1, PC2, PC3, PC4, PC5, PC6, PC7, UART1_RX, UART1_TX
- net labels removed: GPIO_PB3_OUT, GPIO_PB4_OUT, I2C1_SCL, I2C1_SDA, UART_RX, UART_TX
- wire segments 112 -> 170
Other:
- moved on the sheet: C15, C17, C18, C9, D4, D5, P2, R10, R11, R12, R7, R8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
