File: can.sch (KiCad schematic (older format))
At the start: 1 part

Commit message: Basic schematic with temparature and humidity sensor.
Parts:
- removed U?: TJA1042T/3, symbol TJA1042T/3
- added C?: 4n7, symbol C
- added C? (x2): 100n, symbol C
- added JP?: Jumper_NC_Small, symbol Jumper_NC_Small
- added R? (x2): 60, symbol R
- added U?: TJA1042T/3, symbol TJA1042T/3
Connections:
- net labels added: +3.3V, +5V, CANH_IN, CANL_IN, CAN_RX, CAN_STANDBY, CAN_TX, GND
- wire segments 0 -> 26
Changed lines of the file:
@@
 LIBS:74xx
 LIBS:74xgxx
+LIBS:can-node
 LIBS:can-node-cache
 EELAYER 25 0
@@
 $Descr A4 11693 8268
 encoding utf-8
-Sheet 4 4
+Sheet 4 5
 Title ""
 Date ""
@@
 Comment4 ""
 $EndDescr
+Text GLabel 3650 3700 0    60   Input ~ 0
+CAN_TX
+Text GLabel 3650 4000 0    60   Output ~ 0
+CAN_RX
+Wire Wire Line
+	4300 3700 3650 3700
+Wire Wire Line
+	3650 4000 4300 4000
+$Comp
+L GND #PWR?
+U 1 1 57AEDF29
+P 4200 4450
+F 0 "#PWR?" H 4200 4200 50  0001 C CNN
+F 1 "GND" H 4205 4277 50  0000 C CNN
+F 2 "" H 4200 4450 50  0000 C CNN
+F 3 "" H 4200 4450 50  0000 C CNN
+	1    4200 4450
+	1    0    0    -1
+$EndComp
+Wire Wire Line
+	4300 3800 4200 3800
+Wire Wire Line
+	4200 3800 4200 4450
 $Comp
 L TJA1042T/3 U?
-U 1 1 562BA3A0
+U 1 1 57AEDF97
 P 4800 3900
-F 0 "U?" H 4800 3650 60  0000 C CNN
-F 1 "TJA1042T/3" H 4800 4250 60  0000 C CNN
+F 0 "U?" H 4800 4387 60  0000 C CNN
+F 1 "TJA1042T/3" H 4800 4281 60  0000 C CNN
 F 2 "" H 4800 3600 60  0000 C CNN
 F 3 "" H 4800 3600 60  0000 C CNN
@@
 	1    0    0    -1
 $EndComp
+$Comp
+L +5V #PWR?
+U 1 1 57AEED77
+P 4100 3200
+F 0 "#PWR?" H 4100 3050 50  0001 C CNN
+F 1 "+5V" H 4115 3373 50  0000 C CNN
+F 2 "" H 4100 3200 50  0000 C CNN
+F 3 "" H 4100 3200 50  0000 C CNN
+	1    4100 3200
+	1    0    0    -1
+$EndComp
+Wire Wire Line
+	3850 3900 4300 3900
+Wire Wire Line
+	4100 3900 4100 3200
+$Comp
+L +3.3V #PWR?
+U 1 1 57AEEDC2
+P 5400 3200
+F 0 "#PWR?" H 5400 3050 50  0001 C CNN
+F 1 "+3.3V" H 5415 3373 50  0000 C CNN
+F 2 "" H 5400 3200 50  0000 C CNN
+F 3 "" H 5400 3200 50  0000 C CNN
+	1    5400 3200
+	1    0    0    -1
+$EndComp
+Wire Wire Line
+	5400 3200 5400 4100
+Wire Wire Line
+	5400 4000 5300 4000
+Text GLabel 6400 3150 2    60   BiDi ~ 0
+CANH_IN
+Text GLabel 6400 4500 2    60   BiDi ~ 0
+CANL_IN
+$Comp
+L R R?
+U 1 1 57AEEDFE
+P 6250 3650
+F 0 "R?" H 6320 3696 50  0000 L CNN
+F 1 "60" H 6320 3605 50  0000 L CNN
+F 2 "" V 6180 3650 50  0000 C CNN
+F 3 "" H 6250 3650 50  0000 C CNN
+	1    6250 3650
+	1    0    0    -1
+$EndComp
+$Comp
+L R R?
+U 1 1 57AEEEAC
+P 6250 4150
+F 0 "R?" H 6320 4196 50  0000 L CNN
+F 1 "60" H 6320 4105 50  0000 L CNN
+F 2 "" V 6180 4150 50  0000 C CNN
+F 3 "" H 6250 4150 50  0000 C CNN
+	1    6250 4150
+	1    0    0    -1
+$EndComp
+$Comp
+L Jumper_NC_Small JP?
+U 1 1 57AEEED7
+P 6250 3350
+F 0 "JP?" V 6250 3425 50  0000 L CNN
+F 1 "Jumper_NC_Small" H 6260 3290 50  0001 C CNN
+F 2 "" H 6250 3350 50  0000 C CNN
+F 3 "" H 6250 3350 50  0000 C CNN
+	1    6250 3350
+	0    1    1    0
+$EndComp
+Wire Wire Line
+	5750 3150 6400 3150
+Wire Wire Line
+	5750 3150 5750 3800
+Wire Wire Line
+	5750 3800 5300 3800
+Wire Wire Line
+	5300 3900 5750 3900
+Wire Wire Line
+	5750 3900 5750 4500
+Wire Wire Line
+	5750 4500 6400 4500
+Wire Wire Line
+	6250 4300 6250 4500
+Connection ~ 6250 4500
+Wire Wire Line
+	6250 3800 6250 4000
+Wire Wire Line
+	6250 3450 6250 3500
+Wire Wire Line
+	6250 3250 6250 3150
+Connection ~ 6250 3150
+$Comp
+L C C?
+U 1 1 57AEEFE7
+P 5900 4050
+F 0 "C?" H 6015 4096 50  0000 L CNN
+F 1 "4n7" H 6015 4005 50  0000 L CNN
+F 2 "" H 5938 3900 50  0000 C CNN
+F 3 "" H 5900 4050 50  0000 C CNN
+	1    5900 4050
+	1    0    0    -1
+$EndComp
+$Comp
+L GND #PWR?
+U 1 1 57AEF089
+P 5900 4250
+F 0 "#PWR?" H 5900 4000 50  0001 C CNN
+F 1 "GND" H 5905 4077 50  0000 C CNN
+F 2 "" H 5900 4250 50  0000 C CNN
+F 3 "" H 5900 4250 50  0000 C CNN
+	1    5900 4250
+	1    0    0    -1
+$EndComp
+Wire Wire Line
+	5900 4250 5900 4200
+Wire Wire Line
+	5900 3900 5900 3850
+Wire Wire Line
+	5900 3850 6250 3850
+Connection ~ 6250 3850
+Wire Wire Line
+	5300 3700 5300 3350
+Wire Wire Line
+	5300 3350 3650 3350
+Text GLabel 3650 3350 0    60   Input ~ 0
+CAN_STANDBY
+$Comp
+L C C?
+U 1 1 57AF5ACF
+P 3850 4250
+F 0 "C?" H 3965 4296 50  0000 L CNN
+F 1 "100n" H 3965 4205 50  0000 L CNN
+F 2 "" H 3888 4100 50  0000 C CNN
+F 3 "" H 3850 4250 50  0000 C CNN
+	1    3850 4250
+	1    0    0    -1
+$EndComp
+$Comp
+L C C?
+U 1 1 57AF5B9C
+P 5400 4250
+F 0 "C?" H 5515 4296 50  0000 L CNN
+F 1 "100n" H 5515 4205 50  0000 L CNN
+F 2 "" H 5438 4100 50  0000 C CNN
+F 3 "" H 5400 4250 50  0000 C CNN
+	1    5400 4250
+	1    0    0    -1
+$EndComp
+$Comp
+L GND #PWR?
+U 1 1 57AF5C5E
+P 3850 4450
+F 0 "#PWR?" H 3850 4200 50  0001 C CNN
+F 1 "GND" H 3855 4277 50  0000 C CNN
+F 2 "" H 3850 4450 50  0000 C CNN
+F 3 "" H 3850 4450 50  0000 C CNN
+	1    3850 4450
+	1    0    0    -1
+$EndComp
+Wire Wire Line
+	3850 3900 3850 4100
+Connection ~ 4100 3900
+Wire Wire Line
+	3850 4400 3850 4450
+$Comp
+L GND #PWR?
+U 1 1 57AF5CE6
+P 5400 4500
+F 0 "#PWR?" H 5400 4250 50  0001 C CNN
+F 1 "GND" H 5405 4327 50  0000 C CNN
+F 2 "" H 5400 4500 50  0000 C CNN
+F 3 "" H 5400 4500 50  0000 C CNN
+	1    5400 4500
+	1    0    0    -1
+$EndComp
+Wire Wire Line
+	5400 4500 5400 4400
+Connection ~ 5400 4000
 $EndSCHEMATC

Commit message: .
Parts:
- C23, C24: renamed from C?; footprint (none) -> Capacitors_SMD:C_0603_HandSoldering
- R17, R18: renamed from R?; footprint (none) -> Resistors_SMD:R_0603_HandSoldering
- gave numbers to parts that had none: 3
Changed lines of the file:
@@
 	3650 4000 4300 4000
 $Comp
-L GND #PWR?
+L GND #PWR046
 U 1 1 57AEDF29
 P 4200 4450
-F 0 "#PWR?" H 4200 4200 50  0001 C CNN
+F 0 "#PWR046" H 4200 4200 50  0001 C CNN
 F 1 "GND" H 4205 4277 50  0000 C CNN
 F 2 "" H 4200 4450 50  0000 C CNN
@@
 	4200 3800 4200 4450
 $Comp
-L TJA1042T/3 U?
+L TJA1042T/3 U5
 U 1 1 57AEDF97
 P 4800 3900
-F 0 "U?" H 4800 4387 60  0000 C CNN
+F 0 "U5" H 4800 4387 60  0000 C CNN
 F 1 "TJA1042T/3" H 4800 4281 60  0000 C CNN
-F 2 "" H 4800 3600 60  0000 C CNN
+F 2 "" H 4800 3600 60  0001 C CNN
 F 3 "" H 4800 3600 60  0000 C CNN
 	1    4800 3900
@@
 $EndComp
 $Comp
-L +5V #PWR?
+L +5V #PWR047
 U 1 1 57AEED77
 P 4100 3200
-F 0 "#PWR?" H 4100 3050 50  0001 C CNN
+F 0 "#PWR047" H 4100 3050 50  0001 C CNN
 F 1 "+5V" H 4115 3373 50  0000 C CNN
 F 2 "" H 4100 3200 50  0000 C CNN
@@
 	4100 3900 4100 3200
 $Comp
-L +3.3V #PWR?
+L +3.3V #PWR048
 U 1 1 57AEEDC2
 P 5400 3200
-F 0 "#PWR?" H 5400 3050 50  0001 C CNN
+F 0 "#PWR048" H 5400 3050 50  0001 C CNN
 F 1 "+3.3V" H 5415 3373 50  0000 C CNN
 F 2 "" H 5400 3200 50  0000 C CNN
@@
 CANL_IN
 $Comp
-L R R?
+L R R17
 U 1 1 57AEEDFE
 P 6250 3650
-F 0 "R?" H 6320 3696 50  0000 L CNN
+F 0 "R17" H 6320 3696 50  0000 L CNN
 F 1 "60" H 6320 3605 50  0000 L CNN
-F 2 "" V 6180 3650 50  0000 C CNN
+F 2 "Resistors_SMD:R_0603_HandSoldering" V 6180 3650 50  0001 C CNN
 F 3 "" H 6250 3650 50  0000 C CNN
 	1    6250 3650
@@
 $EndComp
 $Comp
-L R R?
+L R R18
 U 1 1 57AEEEAC
 P 6250 4150
-F 0 "R?" H 6320 4196 50  0000 L CNN
+F 0 "R18" H 6320 4196 50  0000 L CNN
 F 1 "60" H 6320 4105 50  0000 L CNN
-F 2 "" V 6180 4150 50  0000 C CNN
+F 2 "Resistors_SMD:R_0603_HandSoldering" V 6180 4150 50  0001 C CNN
 F 3 "" H 6250 4150 50  0000 C CNN
 	1    6250 4150
@@
 $EndComp
 $Comp
-L Jumper_NC_Small JP?
+L Jumper_NC_Small JP1
 U 1 1 57AEEED7
 P 6250 3350
-F 0 "JP?" V 6250 3425 50  0000 L CNN
+F 0 "JP1" V 6250 3425 50  0000 L CNN
 F 1 "Jumper_NC_Small" H 6260 3290 50  0001 C CNN
-F 2 "" H 6250 3350 50  0000 C CNN
+F 2 "" H 6250 3350 50  0001 C CNN
 F 3 "" H 6250 3350 50  0000 C CNN
 	1    6250 3350
@@
 Connection ~ 6250 3150
 $Comp
-L C C?
+L C C25
 U 1 1 57AEEFE7
 P 5900 4050
-F 0 "C?" H 6015 4096 50  0000 L CNN
+F 0 "C25" H 6015 4096 50  0000 L CNN
 F 1 "4n7" H 6015 4005 50  0000 L CNN
-F 2 "" H 5938 3900 50  0000 C CNN
+F 2 "" H 5938 3900 50  0001 C CNN
 F 3 "" H 5900 4050 50  0000 C CNN
 	1    5900 4050
@@
 $EndComp
 $Comp
-L GND #PWR?
+L GND #PWR049
 U 1 1 57AEF089
 P 5900 4250
-F 0 "#PWR?" H 5900 4000 50  0001 C CNN
+F 0 "#PWR049" H 5900 4000 50  0001 C CNN
 F 1 "GND" H 5905 4077 50  0000 C CNN
 F 2 "" H 5900 4250 50  0000 C CNN
@@
 CAN_STANDBY
 $Comp
-L C C?
+L C C23
 U 1 1 57AF5ACF
 P 3850 4250
-F 0 "C?" H 3965 4296 50  0000 L CNN
+F 0 "C23" H 3965 4296 50  0000 L CNN
 F 1 "100n" H 3965 4205 50  0000 L CNN
-F 2 "" H 3888 4100 50  0000 C CNN
+F 2 "Capacitors_SMD:C_0603_HandSoldering" H 3888 4100 50  0001 C CNN
 F 3 "" H 3850 4250 50  0000 C CNN
 	1    3850 4250
@@
 $EndComp
 $Comp
-L C C?
+L C C24
 U 1 1 57AF5B9C
 P 5400 4250
-F 0 "C?" H 5515 4296 50  0000 L CNN
+F 0 "C24" H 5515 4296 50  0000 L CNN
 F 1 "100n" H 5515 4205 50  0000 L CNN
-F 2 "" H 5438 4100 50  0000 C CNN
+F 2 "Capacitors_SMD:C_0603_HandSoldering" H 5438 4100 50  0001 C CNN
 F 3 "" H 5400 4250 50  0000 C CNN
 	1    5400 4250
@@
 $EndComp
 $Comp
-L GND #PWR?
+L GND #PWR050
 U 1 1 57AF5C5E
 P 3850 4450
-F 0 "#PWR?" H 3850 4200 50  0001 C CNN
+F 0 "#PWR050" H 3850 4200 50  0001 C CNN
 F 1 "GND" H 3855 4277 50  0000 C CNN
 F 2 "" H 3850 4450 50  0000 C CNN
@@
 	3850 4400 3850 4450
 $Comp
-L GND #PWR?
+L GND #PWR051
 U 1 1 57AF5CE6
 P 5400 4500
-F 0 "#PWR?" H 5400 4250 50  0001 C CNN
+F 0 "#PWR051" H 5400 4250 50  0001 C CNN
 F 1 "GND" H 5405 4327 50  0000 C CNN
 F 2 "" H 5400 4500 50  0000 C CNN

Commit message: Use TI TCAN334 3.3V CAN transceiver.
Parts:
- removed C24: 100n, Capacitors_SMD:C_0603_HandSoldering, symbol C
- removed U5: TJA1042T/3, symbol TJA1042T/3
- added U?: TCAN334, symbol TCAN334
- R17, R18: value 60 -> 61.9
Connections:
- net labels added: CAN_SHUTDOWN
- net labels removed: +5V
- wire segments 26 -> 29
Other:
- moved on the sheet: C23
Changed lines of the file:
@@
 L GND #PWR046
 U 1 1 57AEDF29
-P 4200 4450
-F 0 "#PWR046" H 4200 4200 50  0001 C CNN
-F 1 "GND" H 4205 4277 50  0000 C CNN
-F 2 "" H 4200 4450 50  0000 C CNN
-F 3 "" H 4200 4450 50  0000 C CNN
-	1    4200 4450
+P 3850 4550
+F 0 "#PWR046" H 3850 4300 50  0001 C CNN
+F 1 "GND" H 3855 4377 50  0000 C CNN
+F 2 "" H 3850 4550 50  0000 C CNN
+F 3 "" H 3850 4550 50  0000 C CNN
+	1    3850 4550
 	1    0    0    -1
 $EndComp
 Wire Wire Line
-	4300 3800 4200 3800
+	4300 3800 3850 3800
 Wire Wire Line
-	4200 3800 4200 4450
-$Comp
-L TJA1042T/3 U5
-U 1 1 57AEDF97
-P 4800 3900
-F 0 "U5" H 4800 4387 60  0000 C CNN
-F 1 "TJA1042T/3" H 4800 4281 60  0000 C CNN
-F 2 "" H 4800 3600 60  0001 C CNN
-F 3 "" H 4800 3600 60  0000 C CNN
-	1    4800 3900
-	1    0    0    -1
-$EndComp
-$Comp
-L +5V #PWR047
-U 1 1 57AEED77
-P 4100 3200
-F 0 "#PWR047" H 4100 3050 50  0001 C CNN
-F 1 "+5V" H 4115 3373 50  0000 C CNN
-F 2 "" H 4100 3200 50  0000 C CNN
-F 3 "" H 4100 3200 50  0000 C CNN
-	1    4100 3200
-	1    0    0    -1
-$EndComp
+	3850 3800 3850 4550
 Wire Wire Line
-	3850 3900 4300 3900
+	4100 3900 4300 3900
 Wire Wire Line
-	4100 3900 4100 3200
+	4100 3900 4100 2950
 $Comp
 L +3.3V #PWR048
 U 1 1 57AEEDC2
-P 5400 3200
-F 0 "#PWR048" H 5400 3050 50  0001 C CNN
-F 1 "+3.3V" H 5415 3373 50  0000 C CNN
-F 2 "" H 5400 3200 50  0000 C CNN
-F 3 "" H 5400 3200 50  0000 C CNN
-	1    5400 3200
+P 4100 2950
+F 0 "#PWR048" H 4100 2800 50  0001 C CNN
+F 1 "+3.3V" H 4115 3123 50  0000 C CNN
+F 2 "" H 4100 2950 50  0000 C CNN
+F 3 "" H 4100 2950 50  0000 C CNN
+	1    4100 2950
 	1    0    0    -1
 $EndComp
-Wire Wire Line
-	5400 3200 5400 4100
-Wire Wire Line
-	5400 4000 5300 4000
 Text GLabel 6400 3150 2    60   BiDi ~ 0
 CANH_IN
@@
 P 6250 3650
 F 0 "R17" H 6320 3696 50  0000 L CNN
-F 1 "60" H 6320 3605 50  0000 L CNN
+F 1 "61.9" H 6320 3605 50  0000 L CNN
 F 2 "Resistors_SMD:R_0603_HandSoldering" V 6180 3650 50  0001 C CNN
 F 3 "" H 6250 3650 50  0000 C CNN
@@
 P 6250 4150
 F 0 "R18" H 6320 4196 50  0000 L CNN
-F 1 "60" H 6320 4105 50  0000 L CNN
+F 1 "61.9" H 6320 4105 50  0000 L CNN
 F 2 "Resistors_SMD:R_0603_HandSoldering" V 6180 4150 50  0001 C CNN
 F 3 "" H 6250 4150 50  0000 C CNN
@@
 $EndComp
 Wire Wire Line
-	5750 3150 6400 3150
+	5750 3150 6250 3150
+Wire Wire Line
+	6250 3150 6400 3150
 Wire Wire Line
 	5750 3150 5750 3800
@@
 	5750 3900 5750 4500
 Wire Wire Line
-	5750 4500 6400 4500
+	5750 4500 6250 4500
+Wire Wire Line
+	6250 4500 6400 4500
 Wire Wire Line
 	6250 4300 6250 4500
 Connection ~ 6250 4500
 Wire Wire Line
-	6250 3800 6250 4000
+	6250 3800 6250 3850
+Wire Wire Line
+	6250 3850 6250 4000
 Wire Wire Line
 	6250 3450 6250 3500
@@
 L C C23
 U 1 1 57AF5ACF
-P 3850 4250
-F 0 "C23" H 3965 4296 50  0000 L CNN
-F 1 "100n" H 3965 4205 50  0000 L CNN
-F 2 "Capacitors_SMD:C_0603_HandSoldering" H 3888 4100 50  0001 C CNN
-F 3 "" H 3850 4250 50  0000 C CNN
-	1    3850 4250
-	1    0    0    -1
-$EndComp
-$Comp
-L C C24
-U 1 1 57AF5B9C
-P 5400 4250
-F 0 "C24" H 5515 4296 50  0000 L CNN
-F 1 "100n" H 5515 4205 50  0000 L CNN
-F 2 "Capacitors_SMD:C_0603_HandSoldering" H 5438 4100 50  0001 C CNN
-F 3 "" H 5400 4250 50  0000 C CNN
-	1    5400 4250
+P 4100 4250
+F 0 "C23" H 4215 4296 50  0000 L CNN
+F 1 "100n" H 4215 4205 50  0000 L CNN
+F 2 "Capacitors_SMD:C_0603_HandSoldering" H 4138 4100 50  0001 C CNN
+F 3 "" H 4100 4250 50  0000 C CNN
+	1    4100 4250
 	1    0    0    -1
 $EndComp
@@
 L GND #PWR050
 U 1 1 57AF5C5E
-P 3850 4450
-F 0 "#PWR050" H 3850 4200 50  0001 C CNN
-F 1 "GND" H 3855 4277 50  0000 C CNN
-F 2 "" H 3850 4450 50  0000 C CNN
-F 3 "" H 3850 4450 50  0000 C CNN
-	1    3850 4450
+P 4100 4550
+F 0 "#PWR050" H 4100 4300 50  0001 C CNN
+F 1 "GND" H 4105 4377 50  0000 C CNN
+F 2 "" H 4100 4550 50  0000 C CNN
+F 3 "" H 4100 4550 50  0000 C CNN
+	1    4100 4550
 	1    0    0    -1
 $EndComp
 Wire Wire Line
-	3850 3900 3850 4100
+	4100 3900 4100 4100
 Connection ~ 4100 3900
 Wire Wire Line
-	3850 4400 3850 4450
+	4100 4400 4100 4550
 $Comp
-L GND #PWR051
-U 1 1 57AF5CE6
-P 5400 4500
-F 0 "#PWR051" H 5400 4250 50  0001 C CNN
-F 1 "GND" H 5405 4327 50  0000 C CNN
-F 2 "" H 5400 4500 50  0000 C CNN
-F 3 "" H 5400 4500 50  0000 C CNN
-	1    5400 4500
+L TCAN334 U?
+U 1 1 57C099EB
+P 4800 3850
+F 0 "U?" H 4800 4287 60  0000 C CNN
+F 1 "TCAN334" H 4800 4181 60  0000 C CNN
+F 2 "" H 4800 3850 60  0000 C CNN
+F 3 "" H 4800 3850 60  0000 C CNN
+	1    4800 3850
 	1    0    0    -1
 $EndComp
+Text GLabel 3650 3150 0    60   Input ~ 0
+CAN_SHUTDOWN
 Wire Wire Line
-	5400 4500 5400 4400
-Connection ~ 5400 4000
+	3650 3150 5400 3150
+Wire Wire Line
+	5400 3150 5400 4000
+Wire Wire Line
+	5400 4000 5300 4000
 $EndSCHEMATC

Commit message: Reset circuit, minor changes
Parts:
- renumbered C25 to C?, C23 to C?, JP1 to JP?, R17 to R?, R18 to R?
Changed lines of the file:
@@
 	3650 4000 4300 4000
 $Comp
-L GND #PWR046
+L GND #PWR?
 U 1 1 57AEDF29
 P 3850 4550
-F 0 "#PWR046" H 3850 4300 50  0001 C CNN
+F 0 "#PWR?" H 3850 4300 50  0001 C CNN
 F 1 "GND" H 3855 4377 50  0000 C CNN
 F 2 "" H 3850 4550 50  0000 C CNN
@@
 	4100 3900 4300 3900
 Wire Wire Line
-	4100 3900 4100 2950
+	4100 2950 4100 4100
 $Comp
-L +3.3V #PWR048
+L +3.3V #PWR?
 U 1 1 57AEEDC2
 P 4100 2950
-F 0 "#PWR048" H 4100 2800 50  0001 C CNN
+F 0 "#PWR?" H 4100 2800 50  0001 C CNN
 F 1 "+3.3V" H 4115 3123 50  0000 C CNN
 F 2 "" H 4100 2950 50  0000 C CNN
@@
 CANL_IN
 $Comp
-L R R17
+L R R?
 U 1 1 57AEEDFE
 P 6250 3650
-F 0 "R17" H 6320 3696 50  0000 L CNN
+F 0 "R?" H 6320 3696 50  0000 L CNN
 F 1 "61.9" H 6320 3605 50  0000 L CNN
 F 2 "Resistors_SMD:R_0603_HandSoldering" V 6180 3650 50  0001 C CNN
@@
 $EndComp
 $Comp
-L R R18
+L R R?
 U 1 1 57AEEEAC
 P 6250 4150
-F 0 "R18" H 6320 4196 50  0000 L CNN
+F 0 "R?" H 6320 4196 50  0000 L CNN
 F 1 "61.9" H 6320 4105 50  0000 L CNN
 F 2 "Resistors_SMD:R_0603_HandSoldering" V 6180 4150 50  0001 C CNN
@@
 $EndComp
 $Comp
-L Jumper_NC_Small JP1
+L Jumper_NC_Small JP?
 U 1 1 57AEEED7
 P 6250 3350
-F 0 "JP1" V 6250 3425 50  0000 L CNN
+F 0 "JP?" V 6250 3425 50  0000 L CNN
 F 1 "Jumper_NC_Small" H 6260 3290 50  0001 C CNN
 F 2 "" H 6250 3350 50  0001 C CNN
@@
 $EndComp
 Wire Wire Line
-	5750 3150 6250 3150
-Wire Wire Line
-	6250 3150 6400 3150
+	5750 3150 6400 3150
 Wire Wire Line
 	5750 3150 5750 3800
@@
 	5750 3900 5750 4500
 Wire Wire Line
-	5750 4500 6250 4500
-Wire Wire Line
-	6250 4500 6400 4500
+	5750 4500 6400 4500
 Wire Wire Line
 	6250 4300 6250 4500
 Connection ~ 6250 4500
 Wire Wire Line
-	6250 3800 6250 3850
-Wire Wire Line
-	6250 3850 6250 4000
+	6250 3800 6250 4000
 Wire Wire Line
 	6250 3450 6250 3500
@@
 Connection ~ 6250 3150
 $Comp
-L C C25
+L C C?
 U 1 1 57AEEFE7
 P 5900 4050
-F 0 "C25" H 6015 4096 50  0000 L CNN
+F 0 "C?" H 6015 4096 50  0000 L CNN
 F 1 "4n7" H 6015 4005 50  0000 L CNN
 F 2 "" H 5938 3900 50  0001 C CNN
@@
 $EndComp
 $Comp
-L GND #PWR049
+L GND #PWR?
 U 1 1 57AEF089
 P 5900 4250
-F 0 "#PWR049" H 5900 4000 50  0001 C CNN
+F 0 "#PWR?" H 5900 4000 50  0001 C CNN
 F 1 "GND" H 5905 4077 50  0000 C CNN
 F 2 "" H 5900 4250 50  0000 C CNN
@@
 CAN_STANDBY
 $Comp
-L C C23
+L C C?
 U 1 1 57AF5ACF
 P 4100 4250
-F 0 "C23" H 4215 4296 50  0000 L CNN
+F 0 "C?" H 4215 4296 50  0000 L CNN
 F 1 "100n" H 4215 4205 50  0000 L CNN
 F 2 "Capacitors_SMD:C_0603_HandSoldering" H 4138 4100 50  0001 C CNN
@@
 $EndComp
 $Comp
-L GND #PWR050
+L GND #PWR?
 U 1 1 57AF5C5E
 P 4100 4550
-F 0 "#PWR050" H 4100 4300 50  0001 C CNN
+F 0 "#PWR?" H 4100 4300 50  0001 C CNN
 F 1 "GND" H 4105 4377 50  0000 C CNN
 F 2 "" H 4100 4550 50  0000 C CNN
@@
 	1    0    0    -1
 $EndComp
-Wire Wire Line
-	4100 3900 4100 4100
 Connection ~ 4100 3900
 Wire Wire Line

Commit message: .
Parts:
- C24: renamed from C?; footprint Capacitors_SMD:C_0603_HandSoldering -> Capacitors_SMD:C_0603
- C25: renamed from C?; footprint (none) -> Capacitors_SMD:C_0603
- R17, R18: renamed from R?; footprint Resistors_SMD:R_0603_HandSoldering -> Resistors_SMD:R_0603
- gave numbers to parts that had none: 2
Changed lines of the file:
@@
 	3650 4000 4300 4000
 $Comp
-L GND #PWR?
+L GND #PWR058
 U 1 1 57AEDF29
 P 3850 4550
-F 0 "#PWR?" H 3850 4300 50  0001 C CNN
+F 0 "#PWR058" H 3850 4300 50  0001 C CNN
 F 1 "GND" H 3855 4377 50  0000 C CNN
 F 2 "" H 3850 4550 50  0000 C CNN
@@
 	4100 2950 4100 4100
 $Comp
-L +3.3V #PWR?
+L +3.3V #PWR059
 U 1 1 57AEEDC2
 P 4100 2950
-F 0 "#PWR?" H 4100 2800 50  0001 C CNN
+F 0 "#PWR059" H 4100 2800 50  0001 C CNN
 F 1 "+3.3V" H 4115 3123 50  0000 C CNN
 F 2 "" H 4100 2950 50  0000 C CNN
@@
 CANL_IN
 $Comp
-L R R?
+L R R17
 U 1 1 57AEEDFE
 P 6250 3650
-F 0 "R?" H 6320 3696 50  0000 L CNN
+F 0 "R17" H 6320 3696 50  0000 L CNN
 F 1 "61.9" H 6320 3605 50  0000 L CNN
-F 2 "Resistors_SMD:R_0603_HandSoldering" V 6180 3650 50  0001 C CNN
+F 2 "Resistors_SMD:R_0603" V 6180 3650 50  0001 C CNN
 F 3 "" H 6250 3650 50  0000 C CNN
 	1    6250 3650
@@
 $EndComp
 $Comp
-L R R?
+L R R18
 U 1 1 57AEEEAC
 P 6250 4150
-F 0 "R?" H 6320 4196 50  0000 L CNN
+F 0 "R18" H 6320 4196 50  0000 L CNN
 F 1 "61.9" H 6320 4105 50  0000 L CNN
-F 2 "Resistors_SMD:R_0603_HandSoldering" V 6180 4150 50  0001 C CNN
+F 2 "Resistors_SMD:R_0603" V 6180 4150 50  0001 C CNN
 F 3 "" H 6250 4150 50  0000 C CNN
 	1    6250 4150
@@
 $EndComp
 $Comp
-L Jumper_NC_Small JP?
+L Jumper_NC_Small JP1
 U 1 1 57AEEED7
 P 6250 3350
-F 0 "JP?" V 6250 3425 50  0000 L CNN
+F 0 "JP1" V 6250 3425 50  0000 L CNN
 F 1 "Jumper_NC_Small" H 6260 3290 50  0001 C CNN
 F 2 "" H 6250 3350 50  0001 C CNN
@@
 Connection ~ 6250 3150
 $Comp
-L C C?
+L C C25
 U 1 1 57AEEFE7
 P 5900 4050
-F 0 "C?" H 6015 4096 50  0000 L CNN
+F 0 "C25" H 6015 4096 50  0000 L CNN
 F 1 "4n7" H 6015 4005 50  0000 L CNN
-F 2 "" H 5938 3900 50  0001 C CNN
+F 2 "Capacitors_SMD:C_0603" H 5938 3900 50  0001 C CNN
 F 3 "" H 5900 4050 50  0000 C CNN
 	1    5900 4050
@@
 $EndComp
 $Comp
-L GND #PWR?
+L GND #PWR060
 U 1 1 57AEF089
 P 5900 4250
-F 0 "#PWR?" H 5900 4000 50  0001 C CNN
+F 0 "#PWR060" H 5900 4000 50  0001 C CNN
 F 1 "GND" H 5905 4077 50  0000 C CNN
 F 2 "" H 5900 4250 50  0000 C CNN
@@
 CAN_STANDBY
 $Comp
-L C C?
+L C C24
 U 1 1 57AF5ACF
 P 4100 4250
-F 0 "C?" H 4215 4296 50  0000 L CNN
+F 0 "C24" H 4215 4296 50  0000 L CNN
 F 1 "100n" H 4215 4205 50  0000 L CNN
-F 2 "Capacitors_SMD:C_0603_HandSoldering" H 4138 4100 50  0001 C CNN
+F 2 "Capacitors_SMD:C_0603" H 4138 4100 50  0001 C CNN
 F 3 "" H 4100 4250 50  0000 C CNN
 	1    4100 4250
@@
 $EndComp
 $Comp
-L GND #PWR?
+L GND #PWR061
 U 1 1 57AF5C5E
 P 4100 4550
-F 0 "#PWR?" H 4100 4300 50  0001 C CNN
+F 0 "#PWR061" H 4100 4300 50  0001 C CNN
 F 1 "GND" H 4105 4377 50  0000 C CNN
 F 2 "" H 4100 4550 50  0000 C CNN
@@
 	4100 4400 4100 4550
 $Comp
-L TCAN334 U?
+L TCAN334 U5
 U 1 1 57C099EB
 P 4800 3850
-F 0 "U?" H 4800 4287 60  0000 C CNN
+F 0 "U5" H 4800 4287 60  0000 C CNN
 F 1 "TCAN334" H 4800 4181 60  0000 C CNN
-F 2 "" H 4800 3850 60  0000 C CNN
+F 2 "" H 4800 3850 60  0001 C CNN
 F 3 "" H 4800 3850 60  0000 C CNN
 	1    4800 3850
