File: can.sch (KiCad schematic (older format))
At the start: 6 parts, among them U5 TCAN334

Commit message: Use LMR16006 DCDC
Parts:
- renumbered C23 to C?, C22 to C?, JP1 to JP?, R16 to R?, R17 to R?, U5 to U?
Changed lines of the file:
@@
 	3650 4000 4300 4000
 $Comp
-L GND #PWR058
+L GND #PWR?
 U 1 1 57AEDF29
 P 3850 4550
-F 0 "#PWR058" H 3850 4300 50  0001 C CNN
+F 0 "#PWR?" H 3850 4300 50  0001 C CNN
 F 1 "GND" H 3855 4377 50  0000 C CNN
 F 2 "" H 3850 4550 50  0000 C CNN
@@
 	4100 2950 4100 4100
 $Comp
-L +3.3V #PWR059
+L +3.3V #PWR?
 U 1 1 57AEEDC2
 P 4100 2950
-F 0 "#PWR059" H 4100 2800 50  0001 C CNN
+F 0 "#PWR?" H 4100 2800 50  0001 C CNN
 F 1 "+3.3V" H 4115 3123 50  0000 C CNN
 F 2 "" H 4100 2950 50  0000 C CNN
@@
 CANL_IN
 $Comp
-L R R16
+L R R?
 U 1 1 57AEEDFE
 P 6250 3650
-F 0 "R16" H 6320 3696 50  0000 L CNN
+F 0 "R?" H 6320 3696 50  0000 L CNN
 F 1 "60.4 1%" H 6320 3605 50  0000 L CNN
 F 2 "Resistors_SMD:R_0603" V 6180 3650 50  0001 C CNN
@@
 $EndComp
 $Comp
-L R R17
+L R R?
 U 1 1 57AEEEAC
 P 6250 4150
-F 0 "R17" H 6320 4196 50  0000 L CNN
+F 0 "R?" H 6320 4196 50  0000 L CNN
 F 1 "60.4 1%" H 6320 4105 50  0000 L CNN
 F 2 "Resistors_SMD:R_0603" V 6180 4150 50  0001 C CNN
@@
 $EndComp
 $Comp
-L Jumper_NC_Small JP1
+L Jumper_NC_Small JP?
 U 1 1 57AEEED7
 P 6250 3350
-F 0 "JP1" V 6250 3425 50  0000 L CNN
+F 0 "JP?" V 6250 3425 50  0000 L CNN
 F 1 "Jumper_NC_Small" H 6260 3290 50  0001 C CNN
 F 2 "" H 6250 3350 50  0001 C CNN
@@
 Connection ~ 6250 3150
 $Comp
-L C C23
+L C C?
 U 1 1 57AEEFE7
 P 5900 4050
-F 0 "C23" H 6015 4096 50  0000 L CNN
+F 0 "C?" H 6015 4096 50  0000 L CNN
 F 1 "4n7" H 6015 4005 50  0000 L CNN
 F 2 "" H 5938 3900 50  0001 C CNN
@@
 $EndComp
 $Comp
-L GND #PWR060
+L GND #PWR?
 U 1 1 57AEF089
 P 5900 4250
-F 0 "#PWR060" H 5900 4000 50  0001 C CNN
+F 0 "#PWR?" H 5900 4000 50  0001 C CNN
 F 1 "GND" H 5905 4077 50  0000 C CNN
 F 2 "" H 5900 4250 50  0000 C CNN
@@
 CAN_STANDBY
 $Comp
-L C C22
+L C C?
 U 1 1 57AF5ACF
 P 4100 4250
-F 0 "C22" H 4215 4296 50  0000 L CNN
+F 0 "C?" H 4215 4296 50  0000 L CNN
 F 1 "100n" H 4215 4205 50  0000 L CNN
 F 2 "" H 4138 4100 50  0001 C CNN
@@
 $EndComp
 $Comp
-L GND #PWR061
+L GND #PWR?
 U 1 1 57AF5C5E
 P 4100 4550
-F 0 "#PWR061" H 4100 4300 50  0001 C CNN
+F 0 "#PWR?" H 4100 4300 50  0001 C CNN
 F 1 "GND" H 4105 4377 50  0000 C CNN
 F 2 "" H 4100 4550 50  0000 C CNN
@@
 	4100 4400 4100 4550
 $Comp
-L TCAN334 U5
+L TCAN334 U?
 U 1 1 57C099EB
 P 4800 3850
-F 0 "U5" H 4800 4287 60  0000 C CNN
+F 0 "U?" H 4800 4287 60  0000 C CNN
 F 1 "TCAN334" H 4800 4181 60  0000 C CNN
 F 2 "" H 4800 3850 60  0001 C CNN

Commit message: Bom
Parts:
- C19, C20: renamed from C?; footprint (none) -> Capacitors_SMD:C_0402
- R13, R14: renamed from R?; footprint Resistors_SMD:R_0603 -> Resistors_SMD:R_0402
- gave numbers to parts that had none: 2
Changed lines of the file:
@@
 	3650 4000 4300 4000
 $Comp
-L GND #PWR?
+L GND #PWR050
 U 1 1 57AEDF29
 P 3850 4550
-F 0 "#PWR?" H 3850 4300 50  0001 C CNN
+F 0 "#PWR050" H 3850 4300 50  0001 C CNN
 F 1 "GND" H 3855 4377 50  0000 C CNN
 F 2 "" H 3850 4550 50  0000 C CNN
@@
 	4100 2950 4100 4100
 $Comp
-L +3.3V #PWR?
+L +3.3V #PWR051
 U 1 1 57AEEDC2
 P 4100 2950
-F 0 "#PWR?" H 4100 2800 50  0001 C CNN
+F 0 "#PWR051" H 4100 2800 50  0001 C CNN
 F 1 "+3.3V" H 4115 3123 50  0000 C CNN
 F 2 "" H 4100 2950 50  0000 C CNN
@@
 CANL_IN
 $Comp
-L R R?
+L R R13
 U 1 1 57AEEDFE
 P 6250 3650
-F 0 "R?" H 6320 3696 50  0000 L CNN
+F 0 "R13" H 6320 3696 50  0000 L CNN
 F 1 "60.4 1%" H 6320 3605 50  0000 L CNN
-F 2 "Resistors_SMD:R_0603" V 6180 3650 50  0001 C CNN
+F 2 "Resistors_SMD:R_0402" V 6180 3650 50  0001 C CNN
 F 3 "" H 6250 3650 50  0000 C CNN
 	1    6250 3650
@@
 $EndComp
 $Comp
-L R R?
+L R R14
 U 1 1 57AEEEAC
 P 6250 4150
-F 0 "R?" H 6320 4196 50  0000 L CNN
+F 0 "R14" H 6320 4196 50  0000 L CNN
 F 1 "60.4 1%" H 6320 4105 50  0000 L CNN
-F 2 "Resistors_SMD:R_0603" V 6180 4150 50  0001 C CNN
+F 2 "Resistors_SMD:R_0402" V 6180 4150 50  0001 C CNN
 F 3 "" H 6250 4150 50  0000 C CNN
 	1    6250 4150
@@
 $EndComp
 $Comp
-L Jumper_NC_Small JP?
+L Jumper_NC_Small JP1
 U 1 1 57AEEED7
 P 6250 3350
-F 0 "JP?" V 6250 3425 50  0000 L CNN
+F 0 "JP1" V 6250 3425 50  0000 L CNN
 F 1 "Jumper_NC_Small" H 6260 3290 50  0001 C CNN
 F 2 "" H 6250 3350 50  0001 C CNN
@@
 Connection ~ 6250 3150
 $Comp
-L C C?
+L C C20
 U 1 1 57AEEFE7
 P 5900 4050
-F 0 "C?" H 6015 4096 50  0000 L CNN
+F 0 "C20" H 6015 4096 50  0000 L CNN
 F 1 "4n7" H 6015 4005 50  0000 L CNN
-F 2 "" H 5938 3900 50  0001 C CNN
+F 2 "Capacitors_SMD:C_0402" H 5938 3900 50  0001 C CNN
 F 3 "" H 5900 4050 50  0000 C CNN
 	1    5900 4050
@@
 $EndComp
 $Comp
-L GND #PWR?
+L GND #PWR052
 U 1 1 57AEF089
 P 5900 4250
-F 0 "#PWR?" H 5900 4000 50  0001 C CNN
+F 0 "#PWR052" H 5900 4000 50  0001 C CNN
 F 1 "GND" H 5905 4077 50  0000 C CNN
 F 2 "" H 5900 4250 50  0000 C CNN
@@
 CAN_STANDBY
 $Comp
-L C C?
+L C C19
 U 1 1 57AF5ACF
 P 4100 4250
-F 0 "C?" H 4215 4296 50  0000 L CNN
+F 0 "C19" H 4215 4296 50  0000 L CNN
 F 1 "100n" H 4215 4205 50  0000 L CNN
-F 2 "" H 4138 4100 50  0001 C CNN
+F 2 "Capacitors_SMD:C_0402" H 4138 4100 50  0001 C CNN
 F 3 "" H 4100 4250 50  0000 C CNN
 	1    4100 4250
@@
 $EndComp
 $Comp
-L GND #PWR?
+L GND #PWR053
 U 1 1 57AF5C5E
 P 4100 4550
-F 0 "#PWR?" H 4100 4300 50  0001 C CNN
+F 0 "#PWR053" H 4100 4300 50  0001 C CNN
 F 1 "GND" H 4105 4377 50  0000 C CNN
 F 2 "" H 4100 4550 50  0000 C CNN
@@
 	4100 4400 4100 4550
 $Comp
-L TCAN334 U?
+L TCAN334 U5
 U 1 1 57C099EB
 P 4800 3850
-F 0 "U?" H 4800 4287 60  0000 C CNN
+F 0 "U5" H 4800 4287 60  0000 C CNN
 F 1 "TCAN334" H 4800 4181 60  0000 C CNN
 F 2 "" H 4800 3850 60  0001 C CNN

Commit message: Finish BOM, assign and add packages, set connectors, minor changes
Parts:
- JP1: footprint (none) -> Pin_Headers:Pin_Header_Straight_1x02
- U5: footprint (none) -> CAN_Node:TI-DCN
Changed lines of the file:
@@
 F 0 "JP1" V 6250 3425 50  0000 L CNN
 F 1 "Jumper_NC_Small" H 6260 3290 50  0001 C CNN
-F 2 "" H 6250 3350 50  0001 C CNN
+F 2 "Pin_Headers:Pin_Header_Straight_1x02" H 6250 3350 50  0001 C CNN
 F 3 "" H 6250 3350 50  0000 C CNN
 	1    6250 3350
@@
 F 0 "U5" H 4800 4287 60  0000 C CNN
 F 1 "TCAN334" H 4800 4181 60  0000 C CNN
-F 2 "" H 4800 3850 60  0001 C CNN
+F 2 "CAN_Node:TI-DCN" H 4800 3850 60  0001 C CNN
 F 3 "" H 4800 3850 60  0000 C CNN
 	1    4800 3850

Commit message: Use solder jumper for optional CAN termination, fix crystal symbol
Parts:
- JP1: footprint Pin_Headers:Pin_Header_Straight_1x02 -> CAN_Node:SolderJumper
Changed lines of the file:
@@
 F 0 "JP1" V 6250 3425 50  0000 L CNN
 F 1 "Jumper_NC_Small" H 6260 3290 50  0001 C CNN
-F 2 "Pin_Headers:Pin_Header_Straight_1x02" H 6250 3350 50  0001 C CNN
+F 2 "CAN_Node:SolderJumper" H 6250 3350 50  0001 C CNN
 F 3 "" H 6250 3350 50  0000 C CNN
 	1    6250 3350

Commit message: Layouting ...
Parts:
- removed JP1: Jumper_NC_Small, CAN_Node:SolderJumper, symbol Jumper_NC_Small
Connections:
- wire segments 25 -> 24
Changed lines of the file:
@@
 	1    0    0    -1
-$EndComp
-$Comp
-L Jumper_NC_Small JP1
-U 1 1 57AEEED7
-P 6250 3350
-F 0 "JP1" V 6250 3425 50  0000 L CNN
-F 1 "Jumper_NC_Small" H 6260 3290 50  0001 C CNN
-F 2 "CAN_Node:SolderJumper" H 6250 3350 50  0001 C CNN
-F 3 "" H 6250 3350 50  0000 C CNN
-	1    6250 3350
-	0    1    1    0
 $EndComp
 Wire Wire Line
@@
 	6250 3800 6250 4000
 Wire Wire Line
-	6250 3450 6250 3500
-Wire Wire Line
-	6250 3250 6250 3150
+	6250 3150 6250 3500
 Connection ~ 6250 3150
 $Comp
