File: can.sch (KiCad schematic (older format))
At the start: 5 parts, among them U5 TCAN334

Commit message: Some modifications to schematic, BOM, start releayout
- add LED display
- change crystal for RTC
- use components that are available at some distributors
Parts:
- U5: footprint CAN_Node:TI-DCN -> can-node:TI-DCN
Changed lines of the file:
@@
 F 0 "U5" H 4800 4287 60  0000 C CNN
 F 1 "TCAN334" H 4800 4181 60  0000 C CNN
-F 2 "CAN_Node:TI-DCN" H 4800 3850 60  0001 C CNN
+F 2 "can-node:TI-DCN" H 4800 3850 60  0001 C CNN
 F 3 "" H 4800 3850 60  0000 C CNN
 	1    4800 3850
