File: connector.sch (KiCad schematic (older format))
At the start: 1 part, among them P3 CONN_01X04

Commit message: Some modifications to schematic, BOM, start releayout
- add LED display
- change crystal for RTC
- use components that are available at some distributors
Parts:
- P3: footprint CAN_Node:WAGO_218-104 -> can-node:WAGO_218-104
Changed lines of the file:
@@
 F 0 "P3" H 5450 4250 50  0000 C CNN
 F 1 "CONN_01X04" V 5550 4000 50  0000 C CNN
-F 2 "CAN_Node:WAGO_218-104" H 5450 4000 50  0001 C CNN
+F 2 "can-node:WAGO_218-104" H 5450 4000 50  0001 C CNN
 F 3 "" H 5450 4000 50  0000 C CNN
 	1    5450 4000
