File: display.sch (KiCad schematic (older format))
At the start: 35 parts, among them Q10 BC807-40, Q11 BC807-40, Q12 BC817-40, Q13 BC817-40, Q14 BC817-40, Q15 BC817-40, Q3 BC817-40, Q4 BC807-40, Q5 BC817-40, Q6 BC807-40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

Commit message: Layouting work
Parts:
- removed Q10, Q11, Q4, Q6, Q8: BC807-40, TO_SOT_Packages_SMD:SOT-23, symbol BC807-40
- removed Q12, Q13, Q14, Q15, Q3, Q5, Q7, Q9: BC817-40, TO_SOT_Packages_SMD:SOT-23, symbol BC817-40
- removed R15, R16, R17, R19, R20, R21, R22, R23, R24, R29, R30, R31, R32: 1k, Resistors_SMD:R_0402, symbol R
- added Q10, Q3, Q4, Q5, Q6, Q7, Q8, Q9: BSS138, TO_SOT_Packages_SMD:SOT-23, symbol BSS138
- added Q11, Q12, Q13, Q14, Q15: BSS84P, TO_SOT_Packages_SMD:SOT-23, symbol BSS84P
Connections:
- wire segments 76 -> 63
