File: display.sch (KiCad schematic (older format))
At the start: 22 parts, among them Q10 BSS138, Q11 BSS84P, Q12 BSS84P, Q13 BSS84P, Q14 BSS84P, Q15 BSS84P, Q3 BSS138, Q4 BSS138, Q5 BSS138, Q6 BSS138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

Commit message: Update for KiCad 5. Assign hand solder foot prints.
Parts:
- AFF1: symbol LTC-4627 -> can-node:LTC-4627
- Q10, Q3, Q4, Q5, Q6, Q7, Q8, Q9: footprint TO_SOT_Packages_SMD:SOT-23 -> TO_SOT_Packages_SMD:SOT-23_Handsoldering; symbol BSS138 -> can-node-rescue:BSS138
- Q11, Q12, Q13, Q14, Q15: footprint TO_SOT_Packages_SMD:SOT-23 -> TO_SOT_Packages_SMD:SOT-23_Handsoldering; symbol BSS84P -> can-node:BSS84P
- R25, R26, R27, R28, R33, R34, R35, R36: footprint Resistors_SMD:R_0402 -> Resistors_SMD:R_0603_HandSoldering; symbol R -> can-node-rescue:R
