File: display.sch (KiCad schematic (older format))
At the start: 22 parts, among them Q10 BSS138, Q11 BSS84P, Q12 BSS84P, Q13 BSS84P, Q14 BSS84P, Q15 BSS84P, Q3 BSS138, Q4 BSS138, Q5 BSS138, Q6 BSS138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

Commit message: Update for KiCad 5.
Parts:
- Q10, Q3, Q4, Q5, Q6, Q7, Q8, Q9: symbol can-node-rescue:BSS138 -> Transistor_FET:BSS138
- R25, R26, R27, R28, R33, R34, R35, R36: symbol can-node-rescue:R -> Device:R
Other:
- moved on the sheet: Q10, Q3, Q4, Q5, Q6, Q7, Q8, Q9
Changed lines of the file:
@@
 PC0
 $Comp
-L can-node-rescue:R R25
+L Device:R R25
 U 1 1 586C588F
 P 4500 4800
@@
 $EndComp
 $Comp
-L can-node-rescue:R R26
+L Device:R R26
 U 1 1 586C5910
 P 5050 5000
@@
 $EndComp
 $Comp
-L can-node-rescue:R R27
+L Device:R R27
 U 1 1 586C5973
 P 5600 5250
@@
 $EndComp
 $Comp
-L can-node-rescue:R R28
+L Device:R R28
 U 1 1 586C598F
 P 6150 5500
@@
 $EndComp
 $Comp
-L can-node-rescue:R R33
+L Device:R R33
 U 1 1 586C59AE
 P 7700 4800
@@
 $EndComp
 $Comp
-L can-node-rescue:R R34
+L Device:R R34
 U 1 1 586C59D0
 P 8250 5050
@@
 $EndComp
 $Comp
-L can-node-rescue:R R35
+L Device:R R35
 U 1 1 586C59F5
 P 8800 5250
@@
 $EndComp
 $Comp
-L can-node-rescue:R R36
+L Device:R R36
 U 1 1 586C5A1D
 P 9350 5500
@@
 	4000 5300 4200 5300
 Wire Wire Line
-	4500 5450 4500 6300
-Wire Wire Line
-	4500 4950 4500 5050
+	4500 5500 4500 6300
+Wire Wire Line
+	4500 4950 4500 5100
 Wire Wire Line
 	4500 4650 4500 4400
@@
 	4000 5800 5300 5800
 Wire Wire Line
-	5050 5700 5050 6300
+	5050 5750 5050 6300
 Wire Wire Line
 	4000 6050 5850 6050
 Wire Wire Line
-	5600 5950 5600 6300
-Wire Wire Line
-	5050 5150 5050 5300
-Wire Wire Line
-	5600 5400 5600 5550
-Wire Wire Line
-	6150 5650 6150 5800
+	5600 6000 5600 6300
+Wire Wire Line
+	5050 5150 5050 5350
+Wire Wire Line
+	5600 5400 5600 5600
+Wire Wire Line
+	6150 5650 6150 5850
 Wire Wire Line
 	5050 4700 5050 4850
@@
 	9350 4350 9350 5350
 Wire Wire Line
-	9350 5650 9350 5800
-Wire Wire Line
-	8800 5550 8800 5400
+	9350 5650 9350 5850
+Wire Wire Line
+	8800 5600 8800 5400
 Wire Wire Line
 	5900 4450 8800 4450
@@
 	5700 4650 5700 4350
 Wire Wire Line
-	7700 4950 7700 5050
-Wire Wire Line
-	8250 5200 8250 5300
-Wire Wire Line
-	9350 6300 9350 6200
-Wire Wire Line
-	8800 6300 8800 5950
-Wire Wire Line
-	8250 6300 8250 5700
-Wire Wire Line
-	7700 6300 7700 5450
+	7700 4950 7700 5100
+Wire Wire Line
+	8250 5200 8250 5350
+Wire Wire Line
+	9350 6300 9350 6250
+Wire Wire Line
+	8800 6300 8800 6000
+Wire Wire Line
+	8250 6300 8250 5750
+Wire Wire Line
+	7700 6300 7700 5500
 Wire Wire Line
 	7200 5300 7400 5300
@@
 PC12
 Wire Wire Line
-	6150 6300 6150 6200
-$Comp
-L can-node-rescue:BSS138 Q3
+	6150 6300 6150 6250
+$Comp
+L Transistor_FET:BSS138 Q3
 U 1 1 586E74D4
-P 4400 5250
+P 4400 5300
 AR Path="/586E74D4" Ref="Q3"  Part="1"
 AR Path="/586C20B6/586E74D4" Ref="Q3"  Part="1"
-F 0 "Q3" H 4591 5296 50  0000 L CNN
-F 1 "BSS138" H 4591 5205 50  0000 L CNN
-F 2 "TO_SOT_Packages_SMD:SOT-23_Handsoldering" H 4600 5175 50  0001 L CIN
-F 3 "" H 4400 5250 50  0000 L CNN
-	1    4400 5250
-	1    0    0    -1
-$EndComp
-$Comp
-L can-node-rescue:BSS138 Q4
+F 0 "Q3" H 4591 5346 50  0000 L CNN
+F 1 "BSS138" H 4591 5255 50  0000 L CNN
+F 2 "TO_SOT_Packages_SMD:SOT-23_Handsoldering" H 4600 5225 50  0001 L CIN
+F 3 "" H 4400 5300 50  0000 L CNN
+	1    4400 5300
+	1    0    0    -1
+$EndComp
+$Comp
+L Transistor_FET:BSS138 Q4
 U 1 1 586E7BEE
-P 4950 5500
+P 4950 5550
 AR Path="/586E7BEE" Ref="Q4"  Part="1"
 AR Path="/586C20B6/586E7BEE" Ref="Q4"  Part="1"
-F 0 "Q4" H 5141 5546 50  0000 L CNN
-F 1 "BSS138" H 5141 5455 50  0000 L CNN
-F 2 "TO_SOT_Packages_SMD:SOT-23_Handsoldering" H 5150 5425 50  0001 L CIN
-F 3 "" H 4950 5500 50  0000 L CNN
-	1    4950 5500
-	1    0    0    -1
-$EndComp
-$Comp
-L can-node-rescue:BSS138 Q5
+F 0 "Q4" H 5141 5596 50  0000 L CNN
+F 1 "BSS138" H 5141 5505 50  0000 L CNN
+F 2 "TO_SOT_Packages_SMD:SOT-23_Handsoldering" H 5150 5475 50  0001 L CIN
+F 3 "" H 4950 5550 50  0000 L CNN
+	1    4950 5550
+	1    0    0    -1
+$EndComp
+$Comp
+L Transistor_FET:BSS138 Q5
 U 1 1 586E7C55
-P 5500 5750
+P 5500 5800
 AR Path="/586E7C55" Ref="Q5"  Part="1"
 AR Path="/586C20B6/586E7C55" Ref="Q5"  Part="1"
-F 0 "Q5" H 5691 5796 50  0000 L CNN
-F 1 "BSS138" H 5691 5705 50  0000 L CNN
-F 2 "TO_SOT_Packages_SMD:SOT-23_Handsoldering" H 5700 5675 50  0001 L CIN
-F 3 "" H 5500 5750 50  0000 L CNN
-	1    5500 5750
-	1    0    0    -1
-$EndComp
-$Comp
-L can-node-rescue:BSS138 Q6
+F 0 "Q5" H 5691 5846 50  0000 L CNN
+F 1 "BSS138" H 5691 5755 50  0000 L CNN
+F 2 "TO_SOT_Packages_SMD:SOT-23_Handsoldering" H 5700 5725 50  0001 L CIN
+F 3 "" H 5500 5800 50  0000 L CNN
+	1    5500 5800
+	1    0    0    -1
+$EndComp
+$Comp
+L Transistor_FET:BSS138 Q6
 U 1 1 586E7CC7
-P 6050 6000
+P 6050 6050
 AR Path="/586E7CC7" Ref="Q6"  Part="1"
 AR Path="/586C20B6/586E7CC7" Ref="Q6"  Part="1"
-F 0 "Q6" H 6241 6046 50  0000 L CNN
-F 1 "BSS138" H 6241 5955 50  0000 L CNN
-F 2 "TO_SOT_Packages_SMD:SOT-23_Handsoldering" H 6250 5925 50  0001 L CIN
-F 3 "" H 6050 6000 50  0000 L CNN
-	1    6050 6000
-	1    0    0    -1
-$EndComp
-$Comp
-L can-node-rescue:BSS138 Q7
+F 0 "Q6" H 6241 6096 50  0000 L CNN
+F 1 "BSS138" H 6241 6005 50  0000 L CNN
+F 2 "TO_SOT_Packages_SMD:SOT-23_Handsoldering" H 6250 5975 50  0001 L CIN
+F 3 "" H 6050 6050 50  0000 L CNN
+	1    6050 6050
+	1    0    0    -1
+$EndComp
+$Comp
+L Transistor_FET:BSS138 Q7
 U 1 1 586E7D3E
-P 7600 5250
+P 7600 5300
 AR Path="/586E7D3E" Ref="Q7"  Part="1"
 AR Path="/586C20B6/586E7D3E" Ref="Q7"  Part="1"
-F 0 "Q7" H 7791 5296 50  0000 L CNN
-F 1 "BSS138" H 7791 5205 50  0000 L CNN
-F 2 "TO_SOT_Packages_SMD:SOT-23_Handsoldering" H 7800 5175 50  0001 L CIN
-F 3 "" H 7600 5250 50  0000 L CNN
-	1    7600 5250
-	1    0    0    -1
-$EndComp
-$Comp
-L can-node-rescue:BSS138 Q8
+F 0 "Q7" H 7791 5346 50  0000 L CNN
+F 1 "BSS138" H 7791 5255 50  0000 L CNN
+F 2 "TO_SOT_Packages_SMD:SOT-23_Handsoldering" H 7800 5225 50  0001 L CIN
+F 3 "" H 7600 5300 50  0000 L CNN
+	1    7600 5300
+	1    0    0    -1
+$EndComp
+$Comp
+L Transistor_FET:BSS138 Q8
 U 1 1 586E7DC6
-P 8150 5500
+P 8150 5550
 AR Path="/586E7DC6" Ref="Q8"  Part="1"
 AR Path="/586C20B6/586E7DC6" Ref="Q8"  Part="1"
-F 0 "Q8" H 8341 5546 50  0000 L CNN
-F 1 "BSS138" H 8341 5455 50  0000 L CNN
-F 2 "TO_SOT_Packages_SMD:SOT-23_Handsoldering" H 8350 5425 50  0001 L CIN
-F 3 "" H 8150 5500 50  0000 L CNN
-	1    8150 5500
-	1    0    0    -1
-$EndComp
-$Comp
-L can-node-rescue:BSS138 Q9
+F 0 "Q8" H 8341 5596 50  0000 L CNN
+F 1 "BSS138" H 8341 5505 50  0000 L CNN
+F 2 "TO_SOT_Packages_SMD:SOT-23_Handsoldering" H 8350 5475 50  0001 L CIN
+F 3 "" H 8150 5550 50  0000 L CNN
+	1    8150 5550
+	1    0    0    -1
+$EndComp
+$Comp
+L Transistor_FET:BSS138 Q9
 U 1 1 586E7E41
-P 8700 5750
+P 8700 5800
 AR Path="/586E7E41" Ref="Q9"  Part="1"
 AR Path="/586C20B6/586E7E41" Ref="Q9"  Part="1"
-F 0 "Q9" H 8891 5796 50  0000 L CNN
-F 1 "BSS138" H 8891 5705 50  0000 L CNN
-F 2 "TO_SOT_Packages_SMD:SOT-23_Handsoldering" H 8900 5675 50  0001 L CIN
-F 3 "" H 8700 5750 50  0000 L CNN
-	1    8700 5750
-	1    0    0    -1
-$EndComp
-$Comp
-L can-node-rescue:BSS138 Q10
+F 0 "Q9" H 8891 5846 50  0000 L CNN
+F 1 "BSS138" H 8891 5755 50  0000 L CNN
+F 2 "TO_SOT_Packages_SMD:SOT-23_Handsoldering" H 8900 5725 50  0001 L CIN
+F 3 "" H 8700 5800 50  0000 L CNN
+	1    8700 5800
+	1    0    0    -1
+$EndComp
+$Comp
+L Transistor_FET:BSS138 Q10
 U 1 1 586E7EBF
-P 9250 6000
+P 9250 6050
 AR Path="/586E7EBF" Ref="Q10"  Part="1"
 AR Path="/586C20B6/586E7EBF" Ref="Q10"  Part="1"
-F 0 "Q10" H 9441 6046 50  0000 L CNN
-F 1 "BSS138" H 9441 5955 50  0000 L CNN
-F 2 "TO_SOT_Packages_SMD:SOT-23_Handsoldering" H 9450 5925 50  0001 L CIN
-F 3 "" H 9250 6000 50  0000 L CNN
-	1    9250 6000
-	1    0    0    -1
-$EndComp
+F 0 "Q10" H 9441 6096 50  0000 L CNN
+F 1 "BSS138" H 9441 6005 50  0000 L CNN
+F 2 "TO_SOT_Packages_SMD:SOT-23_Handsoldering" H 9450 5975 50  0001 L CIN
+F 3 "" H 9250 6050 50  0000 L CNN
+	1    9250 6050
+	1    0    0    -1
+$EndComp

Commit message: Simplify over voltage protection and improve PCB.
- use new KiCad library for some parts
Parts:
- R25, R26, R27, R28, R33, R34, R35, R36: footprint Resistors_SMD:R_0603_HandSoldering -> Resistor_SMD:R_0603_1608Metric_Pad1.05x0.95mm_HandSolder
Changed lines of the file:
@@
 F 0 "R25" H 4570 4846 50  0000 L CNN
 F 1 "120" H 4570 4755 50  0000 L CNN
-F 2 "Resistors_SMD:R_0603_HandSoldering" V 4430 4800 50  0001 C CNN
+F 2 "Resistor_SMD:R_0603_1608Metric_Pad1.05x0.95mm_HandSolder" V 4430 4800 50  0001 C CNN
 F 3 "" H 4500 4800 50  0000 C CNN
 	1    4500 4800
@@
 F 0 "R26" H 5120 5046 50  0000 L CNN
 F 1 "120" H 5120 4955 50  0000 L CNN
-F 2 "Resistors_SMD:R_0603_HandSoldering" V 4980 5000 50  0001 C CNN
+F 2 "Resistor_SMD:R_0603_1608Metric_Pad1.05x0.95mm_HandSolder" V 4980 5000 50  0001 C CNN
 F 3 "" H 5050 5000 50  0000 C CNN
 	1    5050 5000
@@
 F 0 "R27" H 5670 5296 50  0000 L CNN
 F 1 "120" H 5670 5205 50  0000 L CNN
-F 2 "Resistors_SMD:R_0603_HandSoldering" V 5530 5250 50  0001 C CNN
+F 2 "Resistor_SMD:R_0603_1608Metric_Pad1.05x0.95mm_HandSolder" V 5530 5250 50  0001 C CNN
 F 3 "" H 5600 5250 50  0000 C CNN
 	1    5600 5250
@@
 F 0 "R28" H 6220 5546 50  0000 L CNN
 F 1 "120" H 6220 5455 50  0000 L CNN
-F 2 "Resistors_SMD:R_0603_HandSoldering" V 6080 5500 50  0001 C CNN
+F 2 "Resistor_SMD:R_0603_1608Metric_Pad1.05x0.95mm_HandSolder" V 6080 5500 50  0001 C CNN
 F 3 "" H 6150 5500 50  0000 C CNN
 	1    6150 5500
@@
 F 0 "R33" H 7770 4846 50  0000 L CNN
 F 1 "120" H 7770 4755 50  0000 L CNN
-F 2 "Resistors_SMD:R_0603_HandSoldering" V 7630 4800 50  0001 C CNN
+F 2 "Resistor_SMD:R_0603_1608Metric_Pad1.05x0.95mm_HandSolder" V 7630 4800 50  0001 C CNN
 F 3 "" H 7700 4800 50  0000 C CNN
 	1    7700 4800
@@
 F 0 "R34" H 8320 5096 50  0000 L CNN
 F 1 "120" H 8320 5005 50  0000 L CNN
-F 2 "Resistors_SMD:R_0603_HandSoldering" V 8180 5050 50  0001 C CNN
+F 2 "Resistor_SMD:R_0603_1608Metric_Pad1.05x0.95mm_HandSolder" V 8180 5050 50  0001 C CNN
 F 3 "" H 8250 5050 50  0000 C CNN
 	1    8250 5050
@@
 F 0 "R35" H 8870 5296 50  0000 L CNN
 F 1 "120" H 8870 5205 50  0000 L CNN
-F 2 "Resistors_SMD:R_0603_HandSoldering" V 8730 5250 50  0001 C CNN
+F 2 "Resistor_SMD:R_0603_1608Metric_Pad1.05x0.95mm_HandSolder" V 8730 5250 50  0001 C CNN
 F 3 "" H 8800 5250 50  0000 C CNN
 	1    8800 5250
@@
 F 0 "R36" H 9420 5546 50  0000 L CNN
 F 1 "120" H 9420 5455 50  0000 L CNN
-F 2 "Resistors_SMD:R_0603_HandSoldering" V 9280 5500 50  0001 C CNN
+F 2 "Resistor_SMD:R_0603_1608Metric_Pad1.05x0.95mm_HandSolder" V 9280 5500 50  0001 C CNN
 F 3 "" H 9350 5500 50  0000 C CNN
 	1    9350 5500
