File: can-node.sch (KiCad schematic (older format))
At the start: 1 part, among them P2 CONN_01X04

Commit message: Update for KiCad 5.
Parts:
- P2: symbol can-node-rescue:CONN_01X04 -> Connector_Generic:Conn_01x04
Changed lines of the file:
@@
 	2350 2100 2050 2100
 $Comp
-L can-node-rescue:CONN_01X04 P2
+L Connector_Generic:Conn_01x04 P2
 U 1 1 58754CE5
-P 1850 2050
-F 0 "P2" H 1928 2091 50  0000 L CNN
-F 1 "CONN_01X04" H 1928 2000 50  0000 L CNN
-F 2 "can-node:WAGO_218-104" H 1850 2050 50  0001 C CNN
-F 3 "" H 1850 2050 50  0000 C CNN
-	1    1850 2050
+P 1850 2000
+F 0 "P2" H 1928 2041 50  0000 L CNN
+F 1 "CONN_01X04" H 1928 1950 50  0000 L CNN
+F 2 "can-node:WAGO_218-104" H 1850 2000 50  0001 C CNN
+F 3 "" H 1850 2000 50  0000 C CNN
+	1    1850 2000
 	-1   0    0    -1
 $EndComp
